File: KiCAD.kicad_pcb (KiCad board)
At the start: 2 copper layers, 614.7 x 15.2 mm, 233 parts, among them SW1 Esc, SW10 Q, SW100 6, SW101 3, SW102 ., SW103 Tab, SW104 -, SW105 +, SW106 =, SW107 Enter, SW11 A, SW12 F2, SW13 2, SW14 Z, SW15 Win, SW16 W, SW17 S, SW18 F3, SW19 3, SW2 Zen/Han, SW20 X, SW21 Alt, SW22 E, SW23 D, SW24 F4, SW25 4, SW26 C, SW27 R, SW28 F, SW29 5, SW3 Tab, SW30 V, SW31 T, SW32 G, SW33 F5, SW34 6, SW35 B, SW36 Y, SW37 H, SW38 F6, SW39 7, SW4 CaptLock, SW40 N, SW41 SW_MEC_5G_LED, SW42 U, SW43 J, SW44 F7, SW45 8, SW46 M, SW47 I, SW48 K, SW49 F8, SW5 Shift, SW50 9, SW51 ,, SW52 O, SW53 L, SW54 0, SW55 ., SW56 P, SW57 ;, SW58 F9, SW59 -, SW6 Ctrl, SW60 /, SW61 Alt, SW62 @, SW63 :, SW64 F10, SW65 ^, SW66 \, SW67 Win, SW68 [, SW69 ], SW7 F1, SW70 F11, SW71 \, SW72 Fn, SW73 F12, SW74 BS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

Commit message: テンキーを消した。キー軸の上下を逆にした。マイコンを一つ無くした。デバッグ用LEDを無くした。結果PCBnewを作り直すことになった。
Parts:
- D1, D10, D11, D12, D13, D14, D16, D17, D18, D19, D2, D22, D23, D24, D25, D27, D28, D29, D3, D31, D32, D33, D34, D36, D37, D38, D39, D4, D42, D43, D44, D45, D47, D48, D49, D5, D50, D52, D53, D54, D56, D57, D58, D59, D62, D63, D64, D65, D68, D69, D7, D70, D71, D73, D74, D77, D8: moved to F.Cu
- SW1, SW10, SW100, SW101, SW102, SW103, SW104, SW105, SW106, SW107, SW11, SW12, SW13, SW14, SW15, SW16, SW17, SW18, SW19, SW2, SW20, SW21, SW22, SW23, SW24, SW25, SW26, SW27, SW28, SW29, SW3, SW30, SW31, SW32, SW33, SW34, SW35, SW36, SW37, SW38, SW39, SW4, SW40, SW42, SW43, SW44, SW45, SW46, SW47, SW48, SW49, SW5, SW50, SW51, SW52, SW53, SW54, SW55, SW56, SW57, SW58, SW59, SW6, SW60, SW61, SW62, SW63, SW64, SW65, SW66, SW67, SW68, SW69, SW7, SW70, SW71, SW72, SW73, SW74, SW75, SW76, SW77, SW78, SW79, SW8, SW80, SW81, SW82, SW83, SW84, SW85, SW86, SW87, SW88, SW89, SW9, SW90, SW91, SW92, SW93, SW94, SW95, SW96, SW97, SW98, SW99: footprint Cherry_MX_Key_Switch:Cherry_MX_Key_Switch_LED_Pattern1 -> Cherry_MX_Key_Switch:Cherry_MX_Key_Switch_LED_Pattern2
- SW41: value SW_MEC_5G_LED -> Space; footprint Cherry_MX_Key_Switch:Cherry_MX_Key_Switch_LED_Pattern1 -> Cherry_MX_Key_Switch:Cherry_MX_Key_Switch_LED_Pattern2
- moved SW5 455.2 mm to (499.2, 668.8)
- moved SW1 453.9 mm to (499.2, 688.9)
- moved SW2 433.6 mm to (479.1, 709.0)
- moved D104 429.8 mm to (218.1, 791.1), turned to 0 degrees
- moved R4 427.4 mm to (217.9, 797.4), turned to 0 degrees
- moved D106 423.7 mm to (218.1, 794.5), turned to 0 degrees
- moved R3 420.7 mm to (221.9, 797.4), turned to 0 degrees
- moved D105 420.5 mm to (223.9, 787.8), turned to 0 degrees
- moved SW107 420.3 mm to (213.8, 735.8)
- moved D103 417.6 mm to (235.4, 791.1), turned to 0 degrees
- moved SW8 417.3 mm to (479.1, 648.7)
- moved SW12 417.1 mm to (499.2, 648.7)
- moved R2 415.5 mm to (225.9, 797.4), turned to 0 degrees
- moved SW7 415.5 mm to (479.1, 688.9)
- moved D98 414.6 mm to (212.4, 787.8), turned to 0 degrees
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Connections:
- SW1 pad 3: Net-(SW1-Pad3) -> Net-(R1-Pad2)
- SW10 pad 2: Net-(SW10-Pad2) -> GND
- SW10 pad 3: Net-(SW10-Pad3) -> /Line3L
- SW100 pad 2: Net-(SW100-Pad2) -> GND
- SW100 pad 3: Net-(SW100-Pad3) -> /Line4L
- SW101 pad 2: Net-(SW101-Pad2) -> GND
- SW101 pad 3: Net-(SW101-Pad3) -> /Line5L
- SW102 pad 2: Net-(SW102-Pad2) -> GND
- SW102 pad 3: Net-(SW102-Pad3) -> /Line6L
- SW103 pad 2: Net-(SW103-Pad2) -> GND
- SW104 pad 2: Net-(SW104-Pad2) -> GND
- SW105 pad 2: Net-(SW100-Pad3) -> GND
- SW106 pad 2: Net-(SW101-Pad3) -> GND
- SW107 pad 2: Net-(SW102-Pad3) -> GND
- SW11 pad 2: Net-(SW11-Pad2) -> GND
- SW11 pad 3: Net-(SW11-Pad3) -> /Line4L
- SW12 pad 2: Net-(SW12-Pad2) -> GND
- SW12 pad 3: Net-(SW12-Pad3) -> Net-(R1-Pad2)
- SW13 pad 2: Net-(SW13-Pad2) -> GND
- SW13 pad 3: Net-(SW13-Pad3) -> /Line2L
- SW14 pad 2: Net-(SW14-Pad2) -> GND
- SW14 pad 3: Net-(SW14-Pad3) -> /Line5L
- SW15 pad 2: Net-(SW15-Pad2) -> GND
- SW15 pad 3: Net-(SW15-Pad3) -> /Line6L
- SW16 pad 2: Net-(SW10-Pad3) -> GND
- SW16 pad 3: Net-(SW16-Pad3) -> /Line3L
- SW17 pad 2: Net-(SW11-Pad3) -> GND
- SW17 pad 3: Net-(SW17-Pad3) -> /Line4L
- SW18 pad 2: Net-(SW12-Pad3) -> GND
- SW18 pad 3: Net-(SW18-Pad3) -> Net-(R1-Pad2)
- SW19 pad 2: Net-(SW13-Pad3) -> GND
- SW19 pad 3: Net-(SW19-Pad3) -> /Line2L
- SW2 pad 3: Net-(SW2-Pad3) -> /Line2L
- SW20 pad 2: Net-(SW14-Pad3) -> GND
- SW20 pad 3: Net-(SW20-Pad3) -> /Line5L
- SW21 pad 2: Net-(SW15-Pad3) -> GND
- SW21 pad 3: Net-(SW21-Pad3) -> /Line6L
- SW22 pad 2: Net-(SW16-Pad3) -> GND
- SW22 pad 3: Net-(SW22-Pad3) -> /Line3L
- SW23 pad 2: Net-(SW17-Pad3) -> GND
- SW23 pad 3: Net-(SW23-Pad3) -> /Line4L
- SW24 pad 2: Net-(SW18-Pad3) -> GND
- SW24 pad 3: Net-(SW24-Pad3) -> Net-(R1-Pad2)
- SW25 pad 2: Net-(SW19-Pad3) -> GND
- SW25 pad 3: Net-(SW25-Pad3) -> /Line2L
- SW26 pad 2: Net-(SW20-Pad3) -> GND
- SW26 pad 3: Net-(SW26-Pad3) -> /Line5L
- SW27 pad 2: Net-(SW22-Pad3) -> GND
- SW27 pad 3: Net-(SW27-Pad3) -> /Line3L
- SW28 pad 2: Net-(SW23-Pad3) -> GND
- SW28 pad 3: Net-(SW28-Pad3) -> /Line4L
- SW29 pad 2: Net-(SW25-Pad3) -> GND
- SW29 pad 3: Net-(SW29-Pad3) -> /Line2L
- SW3 pad 3: Net-(SW10-Pad2) -> /Line3L
- SW30 pad 2: Net-(SW26-Pad3) -> GND
- SW30 pad 3: Net-(SW30-Pad3) -> /Line5L
- SW31 pad 2: Net-(SW27-Pad3) -> GND
- SW31 pad 3: Net-(SW31-Pad3) -> /Line3L
- SW32 pad 2: Net-(SW28-Pad3) -> GND
- SW32 pad 3: Net-(SW32-Pad3) -> /Line4L
- SW33 pad 2: Net-(SW24-Pad3) -> GND
- SW33 pad 3: Net-(SW33-Pad3) -> Net-(R1-Pad2)
- SW34 pad 2: Net-(SW29-Pad3) -> GND
- SW34 pad 3: Net-(SW34-Pad3) -> /Line2L
- SW35 pad 2: Net-(SW30-Pad3) -> GND
- SW35 pad 3: Net-(SW35-Pad3) -> /Line5L
- SW36 pad 2: Net-(SW31-Pad3) -> GND
- SW36 pad 3: Net-(SW36-Pad3) -> /Line3L
- SW37 pad 2: Net-(SW32-Pad3) -> GND
- SW37 pad 3: Net-(SW37-Pad3) -> /Line4L
- SW38 pad 2: Net-(SW33-Pad3) -> GND
- SW38 pad 3: Net-(SW38-Pad3) -> Net-(R1-Pad2)
- SW39 pad 2: Net-(SW34-Pad3) -> GND
- SW39 pad 3: Net-(SW39-Pad3) -> /Line2L
- SW4 pad 3: Net-(SW11-Pad2) -> /Line4L
- SW40 pad 2: Net-(SW35-Pad3) -> GND
- SW40 pad 3: Net-(SW40-Pad3) -> /Line5L
- SW41 pad 2: Net-(SW21-Pad3) -> GND
- SW41 pad 3: Net-(SW41-Pad3) -> /Line6L
- SW42 pad 2: Net-(SW36-Pad3) -> GND
- SW42 pad 3: Net-(SW42-Pad3) -> /Line3L
- SW43 pad 2: Net-(SW37-Pad3) -> GND
- SW43 pad 3: Net-(SW43-Pad3) -> /Line4L
- SW44 pad 2: Net-(SW38-Pad3) -> GND
- SW44 pad 3: Net-(SW44-Pad3) -> Net-(R1-Pad2)
- SW45 pad 2: Net-(SW39-Pad3) -> GND
- SW45 pad 3: Net-(SW45-Pad3) -> /Line2L
- SW46 pad 2: Net-(SW40-Pad3) -> GND
- SW46 pad 3: Net-(SW46-Pad3) -> /Line5L
- SW47 pad 2: Net-(SW42-Pad3) -> GND
- SW47 pad 3: Net-(SW47-Pad3) -> /Line3L
- SW48 pad 2: Net-(SW43-Pad3) -> GND
- SW48 pad 3: Net-(SW48-Pad3) -> /Line4L
- SW49 pad 2: Net-(SW44-Pad3) -> GND
- SW49 pad 3: Net-(SW49-Pad3) -> Net-(R1-Pad2)
- SW5 pad 3: Net-(SW14-Pad2) -> /Line5L
- SW50 pad 2: Net-(SW45-Pad3) -> GND
- SW50 pad 3: Net-(SW50-Pad3) -> /Line2L
- SW51 pad 2: Net-(SW46-Pad3) -> GND
- SW51 pad 3: Net-(SW51-Pad3) -> /Line5L
- SW52 pad 2: Net-(SW47-Pad3) -> GND
- SW52 pad 3: Net-(SW52-Pad3) -> /Line3L
- SW53 pad 2: Net-(SW48-Pad3) -> GND
- SW53 pad 3: Net-(SW53-Pad3) -> /Line4L
- SW54 pad 2: Net-(SW50-Pad3) -> GND
- SW54 pad 3: Net-(SW54-Pad3) -> /Line2L
- SW55 pad 2: Net-(SW51-Pad3) -> GND
- SW55 pad 3: Net-(SW55-Pad3) -> /Line5L
- SW56 pad 2: Net-(SW52-Pad3) -> GND
- SW56 pad 3: Net-(SW56-Pad3) -> /Line3L
- SW57 pad 2: Net-(SW53-Pad3) -> GND
- SW57 pad 3: Net-(SW57-Pad3) -> /Line4L
- SW58 pad 2: Net-(SW49-Pad3) -> GND
- SW58 pad 3: Net-(SW58-Pad3) -> Net-(R1-Pad2)
- SW59 pad 2: Net-(SW54-Pad3) -> GND
- SW59 pad 3: Net-(SW59-Pad3) -> /Line2L
- SW6 pad 3: Net-(SW6-Pad3) -> /Line6L
- SW60 pad 2: Net-(SW55-Pad3) -> GND
- SW60 pad 3: Net-(SW60-Pad3) -> /Line5L
- SW61 pad 2: Net-(SW41-Pad3) -> GND
- SW61 pad 3: Net-(SW61-Pad3) -> /Line6L
- SW62 pad 2: Net-(SW56-Pad3) -> GND
- SW62 pad 3: Net-(SW62-Pad3) -> /Line3L
- SW63 pad 2: Net-(SW57-Pad3) -> GND
- SW63 pad 3: Net-(SW63-Pad3) -> /Line4L
- SW64 pad 2: Net-(SW58-Pad3) -> GND
- SW64 pad 3: Net-(SW64-Pad3) -> Net-(R1-Pad2)
- SW65 pad 2: Net-(SW59-Pad3) -> GND
- SW65 pad 3: Net-(SW65-Pad3) -> /Line2L
- SW66 pad 2: Net-(SW60-Pad3) -> GND
- SW66 pad 3: Net-(SW66-Pad3) -> /Line5L
- SW67 pad 2: Net-(SW61-Pad3) -> GND
- SW67 pad 3: Net-(SW67-Pad3) -> /Line6L
- SW68 pad 2: Net-(SW62-Pad3) -> GND
- SW68 pad 3: Net-(SW68-Pad3) -> /Line3L
- SW69 pad 2: Net-(SW63-Pad3) -> GND
- SW69 pad 3: Net-(SW69-Pad3) -> /Line4L
- SW7 pad 2: Net-(SW1-Pad3) -> GND
- SW7 pad 3: Net-(SW12-Pad2) -> Net-(R1-Pad2)
- SW70 pad 2: Net-(SW64-Pad3) -> GND
- SW70 pad 3: Net-(SW70-Pad3) -> Net-(R1-Pad2)
- SW71 pad 2: Net-(SW65-Pad3) -> GND
- SW71 pad 3: Net-(SW71-Pad3) -> /Line2L
- SW72 pad 2: Net-(SW67-Pad3) -> GND
- SW72 pad 3: Net-(SW72-Pad3) -> /Line6L
- SW73 pad 2: Net-(SW70-Pad3) -> GND
- SW74 pad 2: Net-(SW71-Pad3) -> GND
- SW74 pad 3: Net-(SW74-Pad3) -> /Line2L
- SW75 pad 2: Net-(SW68-Pad3) -> GND
- SW75 pad 3: Net-(SW75-Pad3) -> /Line3L
- SW76 pad 2: Net-(SW66-Pad3) -> GND
- SW76 pad 3: Net-(SW76-Pad3) -> /Line5L
- SW77 pad 2: Net-(SW72-Pad3) -> GND
- SW77 pad 3: Net-(SW77-Pad3) -> /Line6L
- SW78 pad 2: Net-(SW74-Pad3) -> GND
- SW78 pad 3: Net-(SW78-Pad3) -> /Line2L
- SW79 pad 2: Net-(SW75-Pad3) -> GND
- SW79 pad 3: Net-(SW79-Pad3) -> /Line3L
- SW8 pad 2: Net-(SW2-Pad3) -> GND
- SW8 pad 3: Net-(SW13-Pad2) -> /Line2L
- SW80 pad 2: Net-(SW77-Pad3) -> GND
- SW80 pad 3: Net-(SW80-Pad3) -> /Line6L
- SW81 pad 2: Net-(SW78-Pad3) -> GND
- SW81 pad 3: Net-(SW81-Pad3) -> /Line2L
- SW82 pad 2: Net-(SW79-Pad3) -> GND
- SW82 pad 3: Net-(SW82-Pad3) -> /Line3L
- SW83 pad 2: Net-(SW76-Pad3) -> GND
- SW83 pad 3: Net-(SW83-Pad3) -> /Line5L
- SW84 pad 2: Net-(SW80-Pad3) -> GND
- SW84 pad 3: Net-(SW84-Pad3) -> /Line6L
- SW85 pad 2: Net-(SW81-Pad3) -> GND
- SW85 pad 3: Net-(SW85-Pad3) -> /Line2L
- SW86 pad 2: Net-(SW82-Pad3) -> GND
- SW86 pad 3: Net-(SW86-Pad3) -> /Line3L
- SW87 pad 2: Net-(SW84-Pad3) -> GND
- SW87 pad 3: Net-(SW87-Pad3) -> /Line6L
- SW88 pad 2: Net-(SW85-Pad3) -> GND
- SW88 pad 3: Net-(SW88-Pad3) -> /Line2L
- SW89 pad 2: Net-(SW86-Pad3) -> GND
- SW89 pad 3: Net-(SW89-Pad3) -> /Line3L
- SW9 pad 2: Net-(SW6-Pad3) -> GND
- SW9 pad 3: Net-(SW15-Pad2) -> /Line6L
- SW90 pad 2: Net-(SW69-Pad3) -> GND
- SW90 pad 3: Net-(SW90-Pad3) -> /Line4L
- SW91 pad 2: Net-(SW83-Pad3) -> GND
- SW91 pad 3: Net-(SW91-Pad3) -> /Line5L
- SW92 pad 2: Net-(SW87-Pad3) -> GND
- SW92 pad 3: Net-(SW92-Pad3) -> /Line6L
- SW93 pad 2: Net-(SW88-Pad3) -> GND
- SW93 pad 3: Net-(SW93-Pad3) -> /Line2L
- SW94 pad 2: Net-(SW89-Pad3) -> GND
- SW94 pad 3: Net-(SW94-Pad3) -> /Line3L
- SW95 pad 2: Net-(SW90-Pad3) -> GND
- SW95 pad 3: Net-(SW100-Pad2) -> /Line4L
- SW96 pad 2: Net-(SW91-Pad3) -> GND
- SW96 pad 3: Net-(SW101-Pad2) -> /Line5L
- SW97 pad 2: Net-(SW92-Pad3) -> GND
- SW97 pad 3: Net-(SW102-Pad2) -> /Line6L
- SW98 pad 2: Net-(SW93-Pad3) -> GND
- SW98 pad 3: Net-(SW103-Pad2) -> /Line2L
- SW99 pad 2: Net-(SW94-Pad3) -> GND
- SW99 pad 3: Net-(SW104-Pad2) -> /Line3L
Other:
- board outline removed

Commit message: フットプリントを変えた。
Parts:
- removed D100, D101, D102, D103, D104, D105, D106, D107, D88, D89, D90, D91, D92, D93, D94, D95, D96, D97, D98, D99: 1N4148W, Diode_SMD:D_SOD-123
- removed D108, D109, D110, D111, D112: LED, LED_SMD:LED_0603_1608Metric
- removed R10, R11, R12, R7, R8, R9: R, Resistor_SMD:R_0603_1608Metric
- removed SW100: 6, Cherry_MX_Key_Switch:Cherry_MX_Key_Switch_LED_Pattern2
- removed SW101: 3, Cherry_MX_Key_Switch:Cherry_MX_Key_Switch_LED_Pattern2
- removed SW102: ., Cherry_MX_Key_Switch:Cherry_MX_Key_Switch_LED_Pattern2
- removed SW103: Tab, Cherry_MX_Key_Switch:Cherry_MX_Key_Switch_LED_Pattern2
- removed SW104: -, Cherry_MX_Key_Switch:Cherry_MX_Key_Switch_LED_Pattern2
- removed SW105: +, Cherry_MX_Key_Switch:Cherry_MX_Key_Switch_LED_Pattern2
- removed SW106: =, Cherry_MX_Key_Switch:Cherry_MX_Key_Switch_LED_Pattern2
- removed SW107: Enter, Cherry_MX_Key_Switch:Cherry_MX_Key_Switch_LED_Pattern2
- removed SW89: 7, Cherry_MX_Key_Switch:Cherry_MX_Key_Switch_LED_Pattern2
- removed SW90: 4, Cherry_MX_Key_Switch:Cherry_MX_Key_Switch_LED_Pattern2
- removed SW91: 1, Cherry_MX_Key_Switch:Cherry_MX_Key_Switch_LED_Pattern2
- removed SW92: 0, Cherry_MX_Key_Switch:Cherry_MX_Key_Switch_LED_Pattern2
- removed SW93: /, Cherry_MX_Key_Switch:Cherry_MX_Key_Switch_LED_Pattern2
- removed SW94: 8, Cherry_MX_Key_Switch:Cherry_MX_Key_Switch_LED_Pattern2
- removed SW95: 5, Cherry_MX_Key_Switch:Cherry_MX_Key_Switch_LED_Pattern2
- removed SW96: 2, Cherry_MX_Key_Switch:Cherry_MX_Key_Switch_LED_Pattern2
- removed SW97: 00, Cherry_MX_Key_Switch:Cherry_MX_Key_Switch_LED_Pattern2
- removed SW98: *, Cherry_MX_Key_Switch:Cherry_MX_Key_Switch_LED_Pattern2
- removed SW99: 9, Cherry_MX_Key_Switch:Cherry_MX_Key_Switch_LED_Pattern2
- R1, R2, R3, R4, R5, R6: value R -> 5k
- SW1, SW10, SW11, SW12, SW13, SW14, SW16, SW17, SW18, SW19, SW2, SW20, SW22, SW23, SW24, SW25, SW26, SW27, SW28, SW29, SW30, SW31, SW32, SW33, SW34, SW35, SW36, SW37, SW38, SW39, SW40, SW42, SW43, SW44, SW45, SW46, SW47, SW48, SW49, SW50, SW51, SW52, SW53, SW54, SW55, SW56, SW57, SW58, SW59, SW60, SW62, SW63, SW64, SW65, SW66, SW68, SW69, SW7, SW70, SW71, SW73, SW74, SW78, SW79, SW8, SW80, SW81, SW82, SW83, SW84, SW85, SW86, SW87: footprint Cherry_MX_Key_Switch:Cherry_MX_Key_Switch_LED_Pattern2 -> Button_Switch_Keyboard:SW_Cherry_MX_1.00u_Plate
- SW15, SW3: footprint Cherry_MX_Key_Switch:Cherry_MX_Key_Switch_LED_Pattern2 -> Button_Switch_Keyboard:SW_Cherry_MX_1.50u_Plate
- SW21, SW6, SW61, SW67, SW72, SW77, SW9: footprint Cherry_MX_Key_Switch:Cherry_MX_Key_Switch_LED_Pattern2 -> Button_Switch_Keyboard:SW_Cherry_MX_1.25u_Plate
- SW4, SW41, SW76: footprint Cherry_MX_Key_Switch:Cherry_MX_Key_Switch_LED_Pattern2 -> Button_Switch_Keyboard:SW_Cherry_MX_1.75u_Plate
- SW5: footprint Cherry_MX_Key_Switch:Cherry_MX_Key_Switch_LED_Pattern2 -> Button_Switch_Keyboard:SW_Cherry_MX_2.00u_Plate
- SW75: footprint Cherry_MX_Key_Switch:Cherry_MX_Key_Switch_LED_Pattern2 -> Button_Switch_Keyboard:SW_Cherry_MX_ISOEnter_Plate
- SW88: value BS -> SW_MEC_5G; footprint Cherry_MX_Key_Switch:Cherry_MX_Key_Switch_LED_Pattern2 -> Button_Switch_THT:SW_PUSH_6mm_H5mm
- U1: value Pico -> Master; footprint RaspberryPi_Pico:RPi_Pico_SMD_TH -> Arduino:Sparkfun_Pro_Micro
- U2: value Pico -> Slave; footprint RaspberryPi_Pico:RPi_Pico_SMD_TH -> Arduino:Sparkfun_Pro_Micro
- moved SW26 494.3 mm to (476.1, 290.2)
- moved D82 489.9 mm to (274.8, 302.0)
- moved R4 486.0 mm to (276.2, 314.9)
- moved R5 484.0 mm to (272.2, 314.9)
- moved D79 484.0 mm to (257.6, 310.5)
- moved R6 483.4 mm to (268.2, 314.9)
- moved D87 483.2 mm to (274.8, 312.0)
- moved D83 482.7 mm to (268.1, 305.3)
- moved D69 482.6 mm to (269.1, 302.0)
- moved D80 480.7 mm to (263.3, 310.5)
- moved D21 479.4 mm to (269.1, 312.0)
- moved D86 476.0 mm to (274.8, 308.7)
- moved D84 476.0 mm to (273.9, 305.3)
- moved D76 473.9 mm to (263.3, 313.9)
- moved D85 472.4 mm to (269.1, 308.7)
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Connections:
- D1 pad 1: /Line1S -> Row0
- D10 pad 1: /Line3S -> Row2
- D11 pad 1: /Line4S -> Row3
- D12 pad 1: /Line1S -> Row0
- D13 pad 1: /Line2S -> Row1
- D14 pad 1: /Line5S -> Row4
- D15 pad 1: /Line6S -> Row5
- D16 pad 1: /Line3S -> Row2
- D17 pad 1: /Line4S -> Row3
- D18 pad 1: /Line1S -> Row0
- D19 pad 1: /Line2S -> Row1
- D2 pad 1: /Line2S -> Row1
- D20 pad 1: /Line5S -> Row4
- D21 pad 1: /Line6S -> Row5
- D22 pad 1: /Line3S -> Row2
- D23 pad 1: /Line4S -> Row3
- D24 pad 1: /Line1S -> Row0
- D25 pad 1: /Line2S -> Row1
- D26 pad 1: /Line5S -> Row4
- D27 pad 1: /Line3S -> Row2
- D28 pad 1: /Line4S -> Row3
- D29 pad 1: /Line2S -> Row1
- D3 pad 1: /Line3S -> Row2
- D30 pad 1: /Line5S -> Row4
- D31 pad 1: /Line3S -> Row2
- D32 pad 1: /Line4S -> Row3
- D33 pad 1: /Line1S -> Row0
- D34 pad 1: /Line2S -> Row1
- D35 pad 1: /Line5S -> Row4
- D36 pad 1: /Line3S -> Row2
- D37 pad 1: /Line4S -> Row3
- D38 pad 1: /Line1S -> Row0
- D39 pad 1: /Line2S -> Row1
- D4 pad 1: /Line4S -> Row3
- D40 pad 1: /Line5S -> Row4
- D41 pad 1: /Line6S -> Row5
- D42 pad 1: /Line3S -> Row2
- D43 pad 1: /Line4S -> Row3
- D44 pad 1: /Line1S -> Row0
- D45 pad 1: /Line2S -> Row1
- D46 pad 1: /Line5S -> Row4
- D47 pad 1: /Line3S -> Row2
- D48 pad 1: /Line4S -> Row3
- D49 pad 1: /Line1S -> Row0
- D5 pad 1: /Line5S -> Row4
- D50 pad 1: /Line2S -> Row1
- D51 pad 1: /Line5S -> Row4
- D52 pad 1: /Line3S -> Row2
- D53 pad 1: /Line4S -> Row3
- D54 pad 1: /Line2S -> Row1
- D55 pad 1: /Line5S -> Row4
- D56 pad 1: /Line3S -> Row2
- D57 pad 1: /Line4S -> Row3
- D58 pad 1: /Line1S -> Row0
- D59 pad 1: /Line2 -> Row1
- D6 pad 1: /Line6S -> Row5
- D60 pad 1: /Line5S -> Row4
- D61 pad 1: /Line6S -> Row5
- D62 pad 1: /Line3 -> Row2
- D63 pad 1: /Line4 -> Row3
- D64 pad 1: /Line1 -> Row0
- D65 pad 1: /Line2 -> Row1
- D66 pad 1: /Line5 -> Row4
- D67 pad 1: /Line6 -> Row5
- D68 pad 1: /Line3 -> Row2
- D69 pad 1: /Line4 -> Row3
- D7 pad 1: /Line1S -> Row0
- D70 pad 1: /Line1 -> Row0
- D71 pad 1: /Line2 -> Row1
- D72 pad 1: /Line6 -> Row5
- D73 pad 1: /Line1 -> Row0
- D74 pad 1: /Line4 -> Row3
- D75 pad 1: /Line5 -> Row4
- D76 pad 1: /Line6 -> Row5
- D77 pad 1: /Line3 -> Row2
- D78 pad 1: /Line2 -> Row1
- D79 pad 1: /Line3 -> Row2
- D8 pad 1: /Line2S -> Row1
- D80 pad 1: /Line6 -> Row5
- D81 pad 1: /Line2 -> Row1
- D82 pad 1: /Line3 -> Row2
- D83 pad 1: /Line5 -> Row4
- D84 pad 1: /Line6 -> Row5
- D85 pad 1: /Line2 -> Row1
- D86 pad 1: /Line3 -> Row2
- D87 pad 1: /Line6 -> Row5
- D9 pad 1: /Line6S -> Row5
- R1 pad 1: +5V -> PWM
- R2 pad 1: +5V -> PWM
- R2 pad 2: /Line6L -> Net-(R2-Pad2)
- R3 pad 1: +5V -> PWM
- R3 pad 2: /Line5L -> Net-(R3-Pad2)
- R4 pad 1: +5V -> PWM
- R4 pad 2: /Line4L -> Net-(R4-Pad2)
- R5 pad 1: Net-(D108-Pad1) -> PWM
- R5 pad 2: NumLock_LED -> Net-(R5-Pad2)
- R6 pad 1: +5V -> PWM
- R6 pad 2: /Line3L -> Net-(R6-Pad2)
- SW1 pad 1: /Col1 -> Col0
- SW10 pad 1: /Col2 -> Col1
- SW10 pad 3: /Line3L -> Net-(R3-Pad2)
- SW11 pad 1: /Col2 -> Col1
- SW11 pad 3: /Line4L -> Net-(R2-Pad2)
- SW12 pad 1: /Col3 -> Col2
- SW13 pad 1: /Col3 -> Col2
- SW13 pad 3: /Line2L -> Net-(R5-Pad2)
- SW14 pad 1: /Col2 -> Col1
- SW14 pad 3: /Line5L -> Net-(R4-Pad2)
- SW15 pad 1: /Col3 -> Col2
- SW15 pad 3: /Line6L -> Net-(R4-Pad2)
- SW16 pad 1: /Col3 -> Col2
- SW16 pad 3: /Line3L -> Net-(R3-Pad2)
- SW17 pad 1: /Col3 -> Col2
- SW17 pad 3: /Line4L -> Net-(R2-Pad2)
- SW18 pad 1: /Col4 -> Col3
- SW19 pad 1: /Col4 -> Col3
- SW19 pad 3: /Line2L -> Net-(R5-Pad2)
- SW2 pad 1: /Col1 -> Col0
- SW2 pad 3: /Line2L -> Net-(R1-Pad2)
- SW20 pad 1: /Col3 -> Col2
- SW20 pad 3: /Line5L -> Net-(R4-Pad2)
- SW21 pad 1: /Col4 -> Col3
- SW21 pad 3: /Line6L -> Net-(R4-Pad2)
- SW22 pad 1: /Col4 -> Col3
- SW22 pad 3: /Line3L -> Net-(R3-Pad2)
- SW23 pad 1: /Col4 -> Col3
- SW23 pad 3: /Line4L -> Net-(R2-Pad2)
- SW24 pad 1: /Col5 -> Col4
- SW25 pad 1: /Col5 -> Col4
- SW25 pad 3: /Line2L -> Net-(R5-Pad2)
- SW26 pad 1: /Col4 -> Col3
- SW26 pad 3: /Line5L -> Net-(R4-Pad2)
- SW27 pad 1: /Col5 -> Col4
- SW27 pad 3: /Line3L -> Net-(R3-Pad2)
- SW28 pad 1: /Col5 -> Col4
- SW28 pad 3: /Line4L -> Net-(R2-Pad2)
- SW29 pad 3: /Line2L -> Net-(R5-Pad2)
- SW3 pad 1: /Col1 -> Col0
- SW3 pad 3: /Line3L -> Net-(R3-Pad2)
- SW30 pad 1: /Col5 -> Col4
- SW30 pad 3: /Line5L -> Net-(R4-Pad2)
- SW31 pad 3: /Line3L -> Net-(R3-Pad2)
- SW32 pad 3: /Line4L -> Net-(R2-Pad2)
- SW33 pad 1: /Col6 -> Col5
- SW34 pad 1: /Col6 -> Col5
- SW34 pad 3: /Line2L -> Net-(R5-Pad2)
- SW35 pad 3: /Line5L -> Net-(R4-Pad2)
- SW36 pad 1: /Col6 -> Col5
- SW36 pad 3: /Line3L -> Net-(R3-Pad2)
- SW37 pad 1: /Col6 -> Col5
- SW37 pad 3: /Line4L -> Net-(R2-Pad2)
- SW38 pad 1: /Col7 -> Col6
- SW39 pad 1: /Col7 -> Col6
- SW39 pad 3: /Line2L -> Net-(R5-Pad2)
- SW4 pad 1: /Col1 -> Col0
- SW4 pad 3: /Line4L -> Net-(R2-Pad2)
- SW40 pad 1: /Col6 -> Col5
- SW40 pad 3: /Line5L -> Net-(R4-Pad2)
- SW41 pad 1: /Col6 -> Col5
- SW41 pad 3: /Line6L -> Net-(SW41-Pad3)
- SW42 pad 1: /Col7 -> Col6
- SW42 pad 3: /Line3L -> Net-(R3-Pad2)
- SW43 pad 1: /Col7 -> Col6
- SW43 pad 3: /Line4L -> Net-(R2-Pad2)
- SW44 pad 1: /Col8 -> Col7
- SW45 pad 1: /Col8 -> Col7
- SW45 pad 3: /Line2L -> Net-(R5-Pad2)
- SW46 pad 1: /Col7 -> Col6
- SW46 pad 3: /Line5L -> Net-(R4-Pad2)
- SW47 pad 1: /Col8 -> Col7
- SW47 pad 3: /Line3L -> Net-(R3-Pad2)
- SW48 pad 1: /Col8 -> Col7
- SW48 pad 3: /Line4L -> Net-(R2-Pad2)
- SW49 pad 1: /Col9 -> Col8
- SW5 pad 1: /Col1 -> Col0
- SW5 pad 3: /Line5L -> Net-(R2-Pad2)
- SW50 pad 1: /Col9 -> Col8
- SW50 pad 3: /Line2L -> Net-(R5-Pad2)
- SW51 pad 1: /Col8 -> Col7
- SW51 pad 3: /Line5L -> Net-(R4-Pad2)
- SW52 pad 1: /Col9 -> Col8
- SW52 pad 3: /Line3L -> Net-(R3-Pad2)
- SW53 pad 1: /Col9 -> Col8
- SW53 pad 3: /Line4L -> Net-(R2-Pad2)
- SW54 pad 1: /Col10 -> Col9
- SW54 pad 3: /Line2L -> Net-(R5-Pad2)
- SW55 pad 1: /Col9 -> Col8
- SW55 pad 3: /Line5L -> Net-(R4-Pad2)
- SW56 pad 1: /Col10 -> Col9
- SW56 pad 3: /Line3L -> Net-(R3-Pad2)
- SW57 pad 1: /Col10 -> Col9
- SW57 pad 3: /Line4L -> Net-(R2-Pad2)
- SW58 pad 1: /Col10 -> Col9
- SW59 pad 1: /Col11 -> Col10
- SW59 pad 3: /Line2L -> Net-(R5-Pad2)
- SW6 pad 1: /Col1 -> Col0
- SW6 pad 3: /Line6L -> Net-(R2-Pad2)
- SW60 pad 1: /Col10 -> Col9
- SW60 pad 3: /Line5L -> Net-(R4-Pad2)
- SW61 pad 1: /Col10 -> Col9
- SW61 pad 3: /Line6L -> Net-(SW41-Pad3)
- SW62 pad 1: /Col11 -> Col10
- SW62 pad 3: /Line3L -> Net-(R3-Pad2)
- SW63 pad 1: /Col11 -> Col10
- SW63 pad 3: /Line4L -> Net-(R2-Pad2)
- SW64 pad 1: /Col11 -> Col10
- SW65 pad 1: /Col12 -> Col11
- SW65 pad 3: /Line2L -> Net-(R5-Pad2)
- SW66 pad 1: /Col11 -> Col10
- SW66 pad 3: /Line5L -> Net-(R4-Pad2)
- SW67 pad 1: /Col11 -> Col10
- SW67 pad 3: /Line6L -> Net-(SW41-Pad3)
- SW68 pad 1: /Col12 -> Col11
- SW68 pad 3: /Line3L -> Net-(R3-Pad2)
- SW69 pad 1: /Col12 -> Col11
- SW69 pad 3: /Line4L -> Net-(R2-Pad2)
- SW7 pad 1: /Col2 -> Col1
- SW70 pad 1: /Col12 -> Col11
- SW71 pad 1: /Col13 -> Col12
- SW71 pad 3: /Line2L -> Net-(R5-Pad2)
- SW72 pad 1: /Col12 -> Col11
- SW72 pad 3: /Line6L -> Net-(SW41-Pad3)
- SW73 pad 1: /Col13 -> Col12
- SW74 pad 1: /Col13 -> Col12
- SW74 pad 3: /Line2L -> Net-(R5-Pad2)
- SW75 pad 1: /Col13 -> Col12
- SW75 pad 3: /Line3L -> Net-(R3-Pad2)
- SW76 pad 1: /Col13 -> Col12
- SW76 pad 3: /Line5L -> Net-(R4-Pad2)
- SW77 pad 1: /Col13 -> Col12
- SW77 pad 3: /Line6L -> Net-(SW41-Pad3)
- SW78 pad 1: /Col14 -> Col13
- SW78 pad 3: /Line2L -> Net-(R6-Pad2)
- SW79 pad 1: /Col14 -> Col13
- SW79 pad 3: /Line3L -> Net-(R6-Pad2)
- SW8 pad 1: /Col2 -> Col1
- SW8 pad 3: /Line2L -> Net-(R5-Pad2)
- SW80 pad 1: /Col14 -> Col13
- SW80 pad 3: /Line6L -> Net-(SW41-Pad3)
- SW81 pad 1: /Col15 -> Col14
- SW81 pad 3: /Line2L -> Net-(R6-Pad2)
- SW82 pad 1: /Col15 -> Col14
- SW82 pad 3: /Line3L -> Net-(R6-Pad2)
- SW83 pad 1: /Col15 -> Col14
- SW83 pad 3: /Line5L -> Net-(R6-Pad2)
- SW84 pad 1: /Col15 -> Col14
- SW84 pad 3: /Line6L -> Net-(SW41-Pad3)
- SW85 pad 1: /Col16 -> Col15
- SW85 pad 3: /Line2L -> Net-(R6-Pad2)
- SW86 pad 1: /Col16 -> Col15
- SW86 pad 3: /Line3L -> Net-(R6-Pad2)
- SW87 pad 1: /Col16 -> Col15
- SW87 pad 3: /Line6L -> Net-(R6-Pad2)
- SW88 pad 1: /Col17 -> RST
- SW88 pad 2: GND -> RST
- SW9 pad 1: /Col2 -> Col1
- SW9 pad 3: /Line6L -> Net-(R4-Pad2)
- U1 pad 1: /Col1 -> MasterTX
- U1 pad 10: /Col8 -> Row0
- U1 pad 11: /Col9 -> Col0
- U1 pad 12: /Col10 -> Col1
- U1 pad 13: GND -> PWM
- U1 pad 14: /GPIO10 -> Col2
- U1 pad 15: /GPIO11 -> Col3
- U1 pad 16: /GPIO12 -> Col4
- U1 pad 17: /GPIO13 -> Col5
- U1 pad 18: GND -> Col6
- U1 pad 19: Master_TX -> Col7
- U1 pad 2: /Col2 -> MasterRX
- U1 pad 20: Master_RX -> Col8
- U1 pad 21: NumLock_LED -> VCC
- U1 pad 22: /Line6S -> RST
- U1 pad 24: /Line5S -> +5C
- U1 pad 4: /Col3 -> GND
- U1 pad 5: /Col4 -> Row5
- U1 pad 6: /Col5 -> Row4
- U1 pad 7: /Col6 -> Row3
- U1 pad 8: GND -> Row2
- U1 pad 9: /Col7 -> Row1
- U2 pad 1: /Col11 -> MasterRX
- U2 pad 10: /Col18 -> Col14
- U2 pad 11: /Col19 -> Col15
- U2 pad 12: /Col20 -> Net-(U2-Pad12)
- U2 pad 13: GND -> Net-(U2-Pad13)
- U2 pad 18: GND -> Net-(U2-Pad18)
- U2 pad 19: Master_RX -> Net-(U2-Pad19)
- U2 pad 2: /Col12 -> MasterTX
- U2 pad 20: Master_TX -> Net-(U2-Pad20)
- U2 pad 21: /Line6 -> VCC
- U2 pad 22: /Line5 -> RST
- U2 pad 24: /Line4 -> +5C
- U2 pad 4: /Col13 -> GND
- U2 pad 5: /Col14 -> Col9
- U2 pad 6: /Col15 -> Col10
- U2 pad 7: /Col16 -> Col11
- U2 pad 8: GND -> Col12
- U2 pad 9: /Col17 -> Col13

Commit message: フットプリント配置中
Parts:
- moved U2 858.6 mm to (1018.5, 61.0)
- moved SW75 803.0 mm to (1010.9, 147.3)
- moved SW76 757.7 mm to (1028.7, 251.5)
- moved SW79 743.2 mm to (981.7, 257.8)
- moved SW82 735.4 mm to (1074.4, 259.1)
- moved SW83 686.0 mm to (1041.4, 289.6)
- moved SW72 650.6 mm to (942.3, 289.6)
- moved SW87 587.2 mm to (988.1, 292.1)
- moved SW74 567.9 mm to (927.1, 266.7)
- moved SW70 487.1 mm to (922.0, 231.1)
- moved SW61 401.7 mm to (604.5, 591.8)
- moved SW41 375.7 mm to (497.8, 642.6)
- moved SW5 362.3 mm to (452.1, 612.1)
- moved SW55 320.1 mm to (515.6, 594.4)
- moved SW43 307.0 mm to (393.7, 594.4)
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
Commit message: キーキャップの寸法を確定させないと何も設計できない
Parts:
- moved D10 541.0 mm to (-114.6, 79.1)
- moved D11 541.0 mm to (-120.4, 79.1)
- moved D12 541.0 mm to (-114.6, 75.8)
- moved D13 541.0 mm to (-85.9, 75.8)
- moved D14 541.0 mm to (-126.1, 79.1)
- moved D15 541.0 mm to (-131.9, 79.1)
- moved D16 541.0 mm to (-126.1, 75.8)
- moved D17 541.0 mm to (-131.9, 75.8)
- moved D18 541.0 mm to (-137.6, 79.1)
- moved D19 541.0 mm to (-143.4, 79.1)
- moved D2 541.0 mm to (-91.6, 75.8)
- moved D24 541.0 mm to (-183.6, 72.0)
- moved D25 541.0 mm to (-183.6, 75.3)
- moved D26 541.0 mm to (-143.4, 75.8)
- moved D27 541.0 mm to (-149.1, 79.1)
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
Commit message: Push できる？
Parts:
- SW15: footprint Button_Switch_Keyboard:SW_Cherry_MX_1.50u_Plate -> Button_Switch_Keyboard:SW_Cherry_MX_1.25u_Plate
- moved SW66 848.1 mm to (1080.0, 483.2)
- moved SW63 833.5 mm to (1072.8, 464.2)
- moved SW68 812.1 mm to (1084.5, 445.2)
- moved SW62 786.7 mm to (1065.5, 445.2)
- moved SW58 781.7 mm to (1056.5, 388.2)
- moved SW51 765.1 mm to (1023.0, 483.2)
- moved SW54 756.2 mm to (1037.5, 426.2)
- moved SW59 755.1 mm to (1056.5, 426.2)
- moved SW65 746.6 mm to (1075.5, 426.2)
- moved SW56 714.3 mm to (1046.5, 445.2)
- moved SW57 711.3 mm to (1053.8, 464.2)
- moved SW60 708.5 mm to (1061.0, 483.2)
- moved SW53 708.2 mm to (1034.8, 464.2)
- moved SW52 705.3 mm to (1027.5, 445.2)
- moved SW50 704.7 mm to (1018.5, 426.2)
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
Commit message: PDF を追加
Parts:
- moved D1 528.0 mm to (382.7, 105.3)
- moved D10 528.0 mm to (413.4, 85.4)
- moved D11 528.0 mm to (407.6, 85.4)
- moved D12 528.0 mm to (413.4, 82.0)
- moved D13 528.0 mm to (442.1, 82.0)
- moved D14 528.0 mm to (401.9, 85.4)
- moved D15 528.0 mm to (396.1, 85.4)
- moved D16 528.0 mm to (401.9, 82.0)
- moved D17 528.0 mm to (396.1, 82.0)
- moved D18 528.0 mm to (390.4, 85.4)
- moved D19 528.0 mm to (384.6, 85.4)
- moved D2 528.0 mm to (436.4, 82.0)
- moved D20 528.0 mm to (362.9, 123.1)
- moved D21 528.0 mm to (353.8, 112.5)
- moved D22 528.0 mm to (377.0, 105.3)
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