File: KiCAD.sch (KiCad schematic (older format))
At the start: 233 parts, among them SW1 Esc, SW10 Q, SW100 6, SW101 3, SW102 ., SW103 Tab, SW104 -, SW105 +, SW106 =, SW107 Enter, SW11 A, SW12 F2, SW13 2, SW14 Z, SW15 Win, SW16 W, SW17 S, SW18 F3, SW19 3, SW2 Zen/Han, SW20 X, SW21 Alt, SW22 E, SW23 D, SW24 F4, SW25 4, SW26 C, SW27 R, SW28 F, SW29 5, SW3 Tab, SW30 V, SW31 T, SW32 G, SW33 F5, SW34 6, SW35 B, SW36 Y, SW37 H, SW38 F6, SW39 7, SW4 CaptLock, SW40 N, SW41 SW_MEC_5G_LED, SW42 U, SW43 J, SW44 F7, SW45 8, SW46 M, SW47 I, SW48 K, SW49 F8, SW5 Shift, SW50 9, SW51 ,, SW52 O, SW53 L, SW54 0, SW55 ., SW56 P, SW57 ;, SW58 F9, SW59 -, SW6 Ctrl, SW60 /, SW61 Alt, SW62 @, SW63 :, SW64 F10, SW65 ^, SW66 \\, SW67 Win, SW68 [, SW69 ], SW7 F1, SW70 F11, SW71 \\, SW72 Fn, SW73 F12, SW74 BS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

Commit message: テンキーを消した。キー軸の上下を逆にした。マイコンを一つ無くした。デバッグ用LEDを無くした。結果PCBnewを作り直すことになった。
Parts:
- removed D100, D101, D102, D103, D104, D105, D106, D107, D88, D89, D90, D91, D92, D93, D94, D95, D96, D97, D98, D99: 1N4148W, Diode_SMD:D_SOD-123, symbol Diode:1N4148W
- removed D108, D109, D110, D111, D112: LED, LED_SMD:LED_0603_1608Metric, symbol Device:LED
- removed R10, R11, R12, R5, R8, R9: R, Resistor_SMD:R_0603_1608Metric, symbol Device:R
- removed SW100: 6, Cherry_MX_Key_Switch:Cherry_MX_Key_Switch_LED_Pattern1, symbol Switch:SW_MEC_5G_LED
- removed SW101: 3, Cherry_MX_Key_Switch:Cherry_MX_Key_Switch_LED_Pattern1, symbol Switch:SW_MEC_5G_LED
- removed SW102: ., Cherry_MX_Key_Switch:Cherry_MX_Key_Switch_LED_Pattern1, symbol Switch:SW_MEC_5G_LED
- removed SW103: Tab, Cherry_MX_Key_Switch:Cherry_MX_Key_Switch_LED_Pattern1, symbol Switch:SW_MEC_5G_LED
- removed SW104: -, Cherry_MX_Key_Switch:Cherry_MX_Key_Switch_LED_Pattern1, symbol Switch:SW_MEC_5G_LED
- removed SW105: +, Cherry_MX_Key_Switch:Cherry_MX_Key_Switch_LED_Pattern1, symbol Switch:SW_MEC_5G_LED
- removed SW106: =, Cherry_MX_Key_Switch:Cherry_MX_Key_Switch_LED_Pattern1, symbol Switch:SW_MEC_5G_LED
- removed SW107: Enter, Cherry_MX_Key_Switch:Cherry_MX_Key_Switch_LED_Pattern1, symbol Switch:SW_MEC_5G_LED
- removed SW88: BS, Cherry_MX_Key_Switch:Cherry_MX_Key_Switch_LED_Pattern1, symbol Switch:SW_MEC_5G_LED
- removed SW89: 7, Cherry_MX_Key_Switch:Cherry_MX_Key_Switch_LED_Pattern1, symbol Switch:SW_MEC_5G_LED
- removed SW90: 4, Cherry_MX_Key_Switch:Cherry_MX_Key_Switch_LED_Pattern1, symbol Switch:SW_MEC_5G_LED
- removed SW91: 1, Cherry_MX_Key_Switch:Cherry_MX_Key_Switch_LED_Pattern1, symbol Switch:SW_MEC_5G_LED
- removed SW92: 0, Cherry_MX_Key_Switch:Cherry_MX_Key_Switch_LED_Pattern1, symbol Switch:SW_MEC_5G_LED
- removed SW93: /, Cherry_MX_Key_Switch:Cherry_MX_Key_Switch_LED_Pattern1, symbol Switch:SW_MEC_5G_LED
- removed SW94: 8, Cherry_MX_Key_Switch:Cherry_MX_Key_Switch_LED_Pattern1, symbol Switch:SW_MEC_5G_LED
- removed SW95: 5, Cherry_MX_Key_Switch:Cherry_MX_Key_Switch_LED_Pattern1, symbol Switch:SW_MEC_5G_LED
- removed SW96: 2, Cherry_MX_Key_Switch:Cherry_MX_Key_Switch_LED_Pattern1, symbol Switch:SW_MEC_5G_LED
- removed SW97: 00, Cherry_MX_Key_Switch:Cherry_MX_Key_Switch_LED_Pattern1, symbol Switch:SW_MEC_5G_LED
- removed SW98: *, Cherry_MX_Key_Switch:Cherry_MX_Key_Switch_LED_Pattern1, symbol Switch:SW_MEC_5G_LED
- removed SW99: 9, Cherry_MX_Key_Switch:Cherry_MX_Key_Switch_LED_Pattern1, symbol Switch:SW_MEC_5G_LED
- removed U2: Pico, RaspberryPi_Pico:RPi_Pico_SMD_TH, symbol RaspberryPi_Pico:Pico
- R2, R3, R4, R6, R7: value R -> 100
- SW1, SW10, SW11, SW12, SW13, SW14, SW15, SW16, SW17, SW18, SW19, SW2, SW20, SW21, SW22, SW23, SW24, SW25, SW26, SW27, SW28, SW29, SW3, SW30, SW31, SW32, SW33, SW34, SW35, SW36, SW37, SW38, SW39, SW4, SW40, SW42, SW43, SW44, SW45, SW46, SW47, SW48, SW49, SW5, SW50, SW51, SW52, SW53, SW54, SW55, SW56, SW57, SW58, SW59, SW6, SW60, SW61, SW62, SW63, SW64, SW65, SW66, SW67, SW68, SW69, SW7, SW70, SW71, SW72, SW73, SW74, SW75, SW76, SW77, SW78, SW79, SW8, SW80, SW81, SW82, SW83, SW84, SW85, SW86, SW87, SW9: footprint Cherry_MX_Key_Switch:Cherry_MX_Key_Switch_LED_Pattern1 -> Cherry_MX_Key_Switch:Cherry_MX_Key_Switch_LED_Pattern2
- SW41: value SW_MEC_5G_LED -> Space; footprint Cherry_MX_Key_Switch:Cherry_MX_Key_Switch_LED_Pattern1 -> Cherry_MX_Key_Switch:Cherry_MX_Key_Switch_LED_Pattern2
Connections:
- net labels removed: +3.3V, +3V3, Col17, Col18, Col19, Col20, GPIO10, GPIO11, GPIO12, GPIO13, Line1, Line2, Line3, Line4, Line5, Line6, Master_RX, Master_TX, NumLock_LED
- wire segments 909 -> 918
- no-connect marks 22 -> 9
Other:
- note added: "全てのLEDを並列接続にする。\nカソード側の抵抗値を 100 にする"
- note removed: "マトリックス側の Col とマイコン側の Col が交差しているせいで配線が面倒くさい。\nマイコン側の Col の並び順を入れ替えろ。\n"
- moved on the sheet: R1, R2, R3, R4, R6, R7, U1

Commit message: グローバルラベルにした。
Connections:
- net +5V: no longer R2.1, R3.1, R4.1, R6.1, R7.1
- net GPIO16: now reaches U1.21 (GPIO16)
- net Col1 renamed GPIO0
- net Col10 renamed GPIO9
- net Col11 renamed GPIO10
- net Col12 renamed GPIO11
- net Col13 renamed GPIO12
- net Col14 renamed GPIO13
- net Col15 renamed GPIO14
- net Col16 renamed Gpio15
- net Gpio15: no longer U1.20 (GPIO15)
- net Col2 renamed GPIO1
- net Col3 renamed GPIO2
- net Col4 renamed GPIO3
- net Col5 renamed GPIO4
- net Col6 renamed GPIO5
- net Col7 renamed GPIO6
- net Col8 renamed GPIO7
- net Col9 renamed GPIO8
- net Line1S renamed GPIO22
- net Line2S renamed GPIO21
- net Line3S renamed GPIO20
- net Line4S renamed GPIO19
- net Line5S renamed GPIO18
- net Line6S renamed GPIO17
- new net BackLight: R2.1, R3.1, R4.1, R6.1, R7.1
- new net GPIO15: U1.20 (GPIO15)
- no-connect marks 9 -> 11
Other:
- moved on the sheet: D1, D10, D11, D12, D13, D14, D15, D16, D17, D18, D19, D2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

Commit message: ProMicro
Parts:
- removed R7: 100, Resistor_SMD:R_0603_1608Metric, symbol Device:R
- removed U1: Pico, RaspberryPi_Pico:RPi_Pico_SMD_TH, symbol RaspberryPi_Pico:Pico
- added R5: R, Resistor_SMD:R_0603_1608Metric, symbol Device:R
- added SW88: SW_MEC_5G, Button_Switch_THT:SW_PUSH_6mm_H5mm, symbol Switch:SW_MEC_5G
- added U1: Master, Arduino:Sparkfun_Pro_Micro, symbol Arduino:Sparkfun_Pro_Micro
- added U2: Slave, Arduino:Sparkfun_Pro_Micro, symbol Arduino:Sparkfun_Pro_Micro
- R2, R3, R4, R6: value 100 -> R
Connections:
- net BackLight is gone; now on net PWM: R2.1, R3.1, R4.1, R6.1
- net GND: now also SW88.3 (B), SW88.4 (B), U1.23 (GND), U1.3 (GND), U1.4 (GND), U2.23 (GND), U2.3 (GND), U2.4 (GND)
- net at R1.2, SW1.3 (K), SW12.3 (K)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: now also SW2.3 (K)
- net +5V renamed PWM
- net PWM: now also R5.1, U2.12 (~~D9/A9)
- net GPIO0 renamed Col0
- net Col0: now also U1.11 (D8/A8)
- net GPIO1 renamed Col1
- net Col1: now also U1.12 (~~D9/A9)
- net GPIO10 renamed Col10
- net Col10: now also U2.5 (D2)
- net GPIO11 renamed Col11
- net Col11: now also U2.6 (~~D3)
- net GPIO12 renamed Col12
- net Col12: now also U2.7 (D4/A6)
- net GPIO13 renamed Col13
- net Col13: now also U2.8 (~~D5)
- net GPIO14 renamed Col14
- net Col14: now also U2.9 (~~D6/A7)
- net GPIO17 renamed Row5
- net Row5: now also U1.5 (D2)
- net GPIO18 renamed Row4
- net Row4: now also U1.6 (~~D3)
- net GPIO19 renamed Row3
- net Row3: now also U1.7 (D4/A6)
- net GPIO2 renamed Col2
- net Col2: now also U1.13 (~~D10/A10)
- net GPIO20 renamed Row2
- net Row2: now also U1.8 (~~D5)
- net GPIO21 renamed Row1
- net Row1: now also U1.9 (~~D6/A7)
- net GPIO22 renamed Row0
- net Row0: now also U1.10 (D7)
- net GPIO3 renamed Col3
- net Col3: now also U1.14 (D16)
- net GPIO4 renamed Col4
- net Col4: now also U1.15 (D14)
- net GPIO5 renamed Col5
- net Col5: now also U1.16 (D15)
- net GPIO6 renamed Col6
- net Col6: now also U1.17 (D18/A0)
- net GPIO7 renamed Col7
- net Col7: now also U1.18 (D19/A1)
- net GPIO8 renamed Col8
- net Col8: now also U1.19 (D20/A2)
- net GPIO9 renamed Col9
- net Col9: now also U1.20 (D21/A3)
- net Gpio15 renamed Col15
- net Col15: now also U2.10 (D7)
- net Line2L: no longer names the net of SW13.3 (K), SW19.3 (K), SW25.3 (K), SW29.3 (K), SW34.3 (K), SW39.3 (K), SW45.3 (K), SW50.3 (K), SW54.3 (K), SW59.3 (K), SW65.3 (K), SW71.3 (K), SW74.3 (K), SW8.3 (K)
- net Line2L: now also R5.2; no longer SW2.3 (K), SW78.3 (K), SW81.3 (K), SW85.3 (K)
- net Line3L: no longer names the net of SW10.3 (K), SW16.3 (K), SW22.3 (K), SW27.3 (K), SW3.3 (K), SW31.3 (K), SW36.3 (K), SW42.3 (K), SW47.3 (K), SW52.3 (K), SW56.3 (K), SW62.3 (K), SW68.3 (K), SW75.3 (K)
- net Line3L: now also R3.2; no longer R6.2, SW79.3 (K), SW82.3 (K), SW86.3 (K)
- net Line4L: no longer names the net of SW11.3 (K), SW17.3 (K), SW23.3 (K), SW28.3 (K), SW32.3 (K), SW37.3 (K), SW4.3 (K), SW43.3 (K), SW48.3 (K), SW53.3 (K), SW57.3 (K), SW63.3 (K), SW69.3 (K)
- net Line4L: now also R2.2, SW5.3 (K), SW6.3 (K); no longer R4.2
- net Line5L: no longer names the net of SW14.3 (K), SW20.3 (K), SW26.3 (K), SW30.3 (K), SW35.3 (K), SW40.3 (K), SW46.3 (K), SW51.3 (K), SW55.3 (K), SW60.3 (K), SW66.3 (K), SW76.3 (K)
- net Line5L: now also R4.2, SW15.3 (K), SW21.3 (K), SW9.3 (K); no longer R3.2, SW5.3 (K), SW83.3 (K)
- net Line6L: no longer names the net of SW41.3 (K), SW61.3 (K), SW67.3 (K), SW72.3 (K), SW77.3 (K), SW80.3 (K), SW84.3 (K)
- net Line6L: no longer R2.2, SW15.3 (K), SW21.3 (K), SW6.3 (K), SW87.3 (K), SW9.3 (K)
- new net: R6.2, SW78.3 (K), SW79.3 (K), SW81.3 (K), SW82.3 (K), SW83.3 (K), SW85.3 (K), SW86.3 (K), SW87.3 (K)
- new net +5C: U1.24 (RAW), U2.24 (RAW)
- new net MasterRX: U1.2 (D0/RX), U2.1 (D1/TX)
- new net MasterTX: U1.1 (D1/TX), U2.2 (D0/RX)
- new net RST: SW88.1 (A), SW88.2 (A), U1.22 (RST), U2.22 (RST)
- new net VCC: U1.21 (VCC), U2.21 (VCC)
- no-connect marks 11 -> 9
Other:
- note removed: "全てのLEDを並列接続にする。\nカソード側の抵抗値を 100 にする"
- moved on the sheet: D1, D10, D11, D12, D13, D14, D15, D16, D17, D18, D19, D2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

Commit message: フットプリントを変えた。
Parts:
- R1, R2, R3, R4, R5, R6: value R -> 5k
- SW1, SW10, SW11, SW12, SW13, SW14, SW16, SW17, SW18, SW19, SW2, SW20, SW22, SW23, SW24, SW25, SW26, SW27, SW28, SW29, SW30, SW31, SW32, SW33, SW34, SW35, SW36, SW37, SW38, SW39, SW40, SW42, SW43, SW44, SW45, SW46, SW47, SW48, SW49, SW50, SW51, SW52, SW53, SW54, SW55, SW56, SW57, SW58, SW59, SW60, SW62, SW63, SW64, SW65, SW66, SW68, SW69, SW7, SW70, SW71, SW73, SW74, SW78, SW79, SW8, SW80, SW81, SW82, SW83, SW84, SW85, SW86, SW87: footprint Cherry_MX_Key_Switch:Cherry_MX_Key_Switch_LED_Pattern2 -> Button_Switch_Keyboard:SW_Cherry_MX_1.00u_Plate
- SW15, SW3: footprint Cherry_MX_Key_Switch:Cherry_MX_Key_Switch_LED_Pattern2 -> Button_Switch_Keyboard:SW_Cherry_MX_1.50u_Plate
- SW21, SW6, SW61, SW67, SW72, SW77, SW9: footprint Cherry_MX_Key_Switch:Cherry_MX_Key_Switch_LED_Pattern2 -> Button_Switch_Keyboard:SW_Cherry_MX_1.25u_Plate
- SW4, SW41, SW76: footprint Cherry_MX_Key_Switch:Cherry_MX_Key_Switch_LED_Pattern2 -> Button_Switch_Keyboard:SW_Cherry_MX_1.75u_Plate
- SW5: footprint Cherry_MX_Key_Switch:Cherry_MX_Key_Switch_LED_Pattern2 -> Button_Switch_Keyboard:SW_Cherry_MX_2.00u_Plate
- SW75: footprint Cherry_MX_Key_Switch:Cherry_MX_Key_Switch_LED_Pattern2 -> Button_Switch_Keyboard:SW_Cherry_MX_ISOEnter_Plate
Connections:
- net Col10: now also U2.6 (~~D3); no longer U2.5 (D2)
- net Col11: now also U2.7 (D4/A6); no longer U2.6 (~~D3)
- net Col12: now also U2.8 (~~D5); no longer U2.7 (D4/A6)
- net Col13: now also U2.9 (~~D6/A7); no longer U2.8 (~~D5)
- net Col14: now also U2.10 (D7); no longer U2.9 (~~D6/A7)
- net Col15: now also U2.11 (D8/A8); no longer U2.10 (D7)
- net Col2: now also U1.14 (D16); no longer U1.13 (~~D10/A10)
- net Col3: now also U1.15 (D14); no longer U1.14 (D16)
- net Col4: now also U1.16 (D15); no longer U1.15 (D14)
- net Col5: now also U1.17 (D18/A0); no longer U1.16 (D15)
- net Col6: now also U1.18 (D19/A1); no longer U1.17 (D18/A0)
- net Col7: now also U1.19 (D20/A2); no longer U1.18 (D19/A1)
- net Col8: now also U1.20 (D21/A3); no longer U1.19 (D20/A2)
- net Col9: now also U2.5 (D2); no longer U1.20 (D21/A3)
- net PWM: now also U1.13 (~~D10/A10); no longer U2.12 (~~D9/A9)

Commit message: キーキャップの寸法を確定させないと何も設計できない
Parts:
- U1, U2: symbol Arduino:Sparkfun_Pro_Micro -> KiCAD-rescue:Sparkfun_Pro_Micro-Arduino
Changed lines of the file:
@@
 Col12
 $Comp
-L Arduino:Sparkfun_Pro_Micro U1
+L KiCAD-rescue:Sparkfun_Pro_Micro-Arduino U1
 U 1 1 61433DA9
 P 2950 6050
@@
 Connection ~ 16850 7650
 $Comp
-L Arduino:Sparkfun_Pro_Micro U2
+L KiCAD-rescue:Sparkfun_Pro_Micro-Arduino U2
 U 1 1 63808FF3
 P 5500 6050

Commit message: PDF を追加
Parts:
- SW15: footprint Button_Switch_Keyboard:SW_Cherry_MX_1.50u_Plate -> Button_Switch_Keyboard:SW_Cherry_MX_1.25u_Plate
Changed lines of the file:
@@
 F 0 "SW15" H 4500 14235 50  0000 C CNN
 F 1 "Win" H 4500 14144 50  0000 C CNN
-F 2 "Button_Switch_Keyboard:SW_Cherry_MX_1.50u_Plate" H 4500 14150 50  0001 C CNN
+F 2 "Button_Switch_Keyboard:SW_Cherry_MX_1.25u_Plate" H 4500 14150 50  0001 C CNN
 F 3 "http://www.apem.com/int/index.php?controller=attachment&id_attachment=488" H 4500 14150 50  0001 C CNN
 	1    4500 13850
