File: pcb/main/KiCAD.sch (KiCad schematic (older format))
At the start: 183 parts, among them SW1 Esc, SW10 Q, SW11 A, SW12 F2, SW13 2, SW14 Z, SW15 Win, SW16 W, SW17 S, SW18 F3, SW19 3, SW2 Zen/Han, SW20 X, SW21 Alt, SW22 E, SW23 D, SW24 F4, SW25 4, SW26 C, SW27 R, SW28 F, SW29 5, SW3 Tab, SW30 V, SW31 T, SW32 G, SW33 F5, SW34 6, SW35 B, SW36 Y, SW37 H, SW38 F6, SW39 7, SW4 CaptLock, SW40 N, SW41 Space, SW42 U, SW43 J, SW44 F7, SW45 8, SW46 M, SW47 I, SW48 K, SW49 F8, SW5 Shift, SW50 9, SW51 ,, SW52 O, SW53 L, SW54 0, SW55 ., SW56 P, SW57 ;, SW58 F9, SW59 -, SW6 Ctrl, SW60 /, SW61 Alt, SW62 @, SW63 :, SW64 F10, SW65 ^, SW66 \\, SW67 Win, SW68 [, SW69 ], SW7 F1, SW70 F11, SW71 \\, SW72 Fn, SW73 F12, SW74 BS, SW75 Enter, SW76 Shift, SW77 Ctrl, SW78 PrtSc, SW79 Delete, SW8 1, SW80 Left, SW81 Home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

Commit message: とりあえず完成
Parts:
- removed D1, D10, D11, D12, D13, D14, D15, D16, D17, D18, D19, D2, D20, D21, D22, D23, D24, D25, D26, D27, D28, D29, D3, D30, D31, D32, D33, D34, D35, D36, D37, D38, D39, D4, D40, D41, D42, D43, D44, D45, D46, D47, D48, D49, D5, D50, D51, D52, D53, D54, D55, D56, D57, D58, D59, D6, D60, D61, D62, D63, D64, D65, D66, D67, D68, D69, D7, D70, D71, D72, D73, D74, D75, D76, D77, D78, D79, D8, D80, D81, D82, D83, D84, D85, D86, D87, D9: 1N4148W, Diode_SMD:D_SOD-123, symbol Diode:1N4148W
- removed SW1: Esc, Button_Switch_Keyboard:SW_Cherry_MX_1.00u_Plate, symbol Switch:SW_MEC_5G_LED
- removed SW10: Q, Button_Switch_Keyboard:SW_Cherry_MX_1.00u_Plate, symbol Switch:SW_MEC_5G_LED
- removed SW11: A, Button_Switch_Keyboard:SW_Cherry_MX_1.00u_Plate, symbol Switch:SW_MEC_5G_LED
- removed SW12: F2, Button_Switch_Keyboard:SW_Cherry_MX_1.00u_Plate, symbol Switch:SW_MEC_5G_LED
- removed SW13: 2, Button_Switch_Keyboard:SW_Cherry_MX_1.00u_Plate, symbol Switch:SW_MEC_5G_LED
- removed SW14: Z, Button_Switch_Keyboard:SW_Cherry_MX_1.00u_Plate, symbol Switch:SW_MEC_5G_LED
- removed SW15, SW67: Win, Button_Switch_Keyboard:SW_Cherry_MX_1.25u_Plate, symbol Switch:SW_MEC_5G_LED
- removed SW16: W, Button_Switch_Keyboard:SW_Cherry_MX_1.00u_Plate, symbol Switch:SW_MEC_5G_LED
- removed SW17: S, Button_Switch_Keyboard:SW_Cherry_MX_1.00u_Plate, symbol Switch:SW_MEC_5G_LED
- removed SW18: F3, Button_Switch_Keyboard:SW_Cherry_MX_1.00u_Plate, symbol Switch:SW_MEC_5G_LED
- removed SW19: 3, Button_Switch_Keyboard:SW_Cherry_MX_1.00u_Plate, symbol Switch:SW_MEC_5G_LED
- removed SW2: Zen/Han, Button_Switch_Keyboard:SW_Cherry_MX_1.00u_Plate, symbol Switch:SW_MEC_5G_LED
- removed SW20: X, Button_Switch_Keyboard:SW_Cherry_MX_1.00u_Plate, symbol Switch:SW_MEC_5G_LED
- removed SW21, SW61: Alt, Button_Switch_Keyboard:SW_Cherry_MX_1.25u_Plate, symbol Switch:SW_MEC_5G_LED
- removed SW22: E, Button_Switch_Keyboard:SW_Cherry_MX_1.00u_Plate, symbol Switch:SW_MEC_5G_LED
- removed SW23: D, Button_Switch_Keyboard:SW_Cherry_MX_1.00u_Plate, symbol Switch:SW_MEC_5G_LED
- removed SW24: F4, Button_Switch_Keyboard:SW_Cherry_MX_1.00u_Plate, symbol Switch:SW_MEC_5G_LED
- removed SW25: 4, Button_Switch_Keyboard:SW_Cherry_MX_1.00u_Plate, symbol Switch:SW_MEC_5G_LED
- removed SW26: C, Button_Switch_Keyboard:SW_Cherry_MX_1.00u_Plate, symbol Switch:SW_MEC_5G_LED
- removed SW27: R, Button_Switch_Keyboard:SW_Cherry_MX_1.00u_Plate, symbol Switch:SW_MEC_5G_LED
- removed SW28: F, Button_Switch_Keyboard:SW_Cherry_MX_1.00u_Plate, symbol Switch:SW_MEC_5G_LED
- removed SW29: 5, Button_Switch_Keyboard:SW_Cherry_MX_1.00u_Plate, symbol Switch:SW_MEC_5G_LED
- removed SW3: Tab, Button_Switch_Keyboard:SW_Cherry_MX_1.50u_Plate, symbol Switch:SW_MEC_5G_LED
- removed SW30: V, Button_Switch_Keyboard:SW_Cherry_MX_1.00u_Plate, symbol Switch:SW_MEC_5G_LED
- removed SW31: T, Button_Switch_Keyboard:SW_Cherry_MX_1.00u_Plate, symbol Switch:SW_MEC_5G_LED
- removed SW32: G, Button_Switch_Keyboard:SW_Cherry_MX_1.00u_Plate, symbol Switch:SW_MEC_5G_LED
- removed SW33: F5, Button_Switch_Keyboard:SW_Cherry_MX_1.00u_Plate, symbol Switch:SW_MEC_5G_LED
- removed SW34: 6, Button_Switch_Keyboard:SW_Cherry_MX_1.00u_Plate, symbol Switch:SW_MEC_5G_LED
- removed SW35: B, Button_Switch_Keyboard:SW_Cherry_MX_1.00u_Plate, symbol Switch:SW_MEC_5G_LED
- removed SW36: Y, Button_Switch_Keyboard:SW_Cherry_MX_1.00u_Plate, symbol Switch:SW_MEC_5G_LED
- removed SW37: H, Button_Switch_Keyboard:SW_Cherry_MX_1.00u_Plate, symbol Switch:SW_MEC_5G_LED
- removed SW38: F6, Button_Switch_Keyboard:SW_Cherry_MX_1.00u_Plate, symbol Switch:SW_MEC_5G_LED
- removed SW39: 7, Button_Switch_Keyboard:SW_Cherry_MX_1.00u_Plate, symbol Switch:SW_MEC_5G_LED
- removed SW4: CaptLock, Button_Switch_Keyboard:SW_Cherry_MX_1.75u_Plate, symbol Switch:SW_MEC_5G_LED
- removed SW40: N, Button_Switch_Keyboard:SW_Cherry_MX_1.00u_Plate, symbol Switch:SW_MEC_5G_LED
- removed SW41: Space, Button_Switch_Keyboard:SW_Cherry_MX_1.75u_Plate, symbol Switch:SW_MEC_5G_LED
- removed SW42: U, Button_Switch_Keyboard:SW_Cherry_MX_1.00u_Plate, symbol Switch:SW_MEC_5G_LED
- removed SW43: J, Button_Switch_Keyboard:SW_Cherry_MX_1.00u_Plate, symbol Switch:SW_MEC_5G_LED
- removed SW44: F7, Button_Switch_Keyboard:SW_Cherry_MX_1.00u_Plate, symbol Switch:SW_MEC_5G_LED
- removed SW45: 8, Button_Switch_Keyboard:SW_Cherry_MX_1.00u_Plate, symbol Switch:SW_MEC_5G_LED
- removed SW46: M, Button_Switch_Keyboard:SW_Cherry_MX_1.00u_Plate, symbol Switch:SW_MEC_5G_LED
- removed SW47: I, Button_Switch_Keyboard:SW_Cherry_MX_1.00u_Plate, symbol Switch:SW_MEC_5G_LED
- removed SW48: K, Button_Switch_Keyboard:SW_Cherry_MX_1.00u_Plate, symbol Switch:SW_MEC_5G_LED
- removed SW49: F8, Button_Switch_Keyboard:SW_Cherry_MX_1.00u_Plate, symbol Switch:SW_MEC_5G_LED
- removed SW5: Shift, Button_Switch_Keyboard:SW_Cherry_MX_2.00u_Plate, symbol Switch:SW_MEC_5G_LED
- removed SW50: 9, Button_Switch_Keyboard:SW_Cherry_MX_1.00u_Plate, symbol Switch:SW_MEC_5G_LED
- removed SW51: ,, Button_Switch_Keyboard:SW_Cherry_MX_1.00u_Plate, symbol Switch:SW_MEC_5G_LED
- removed SW52: O, Button_Switch_Keyboard:SW_Cherry_MX_1.00u_Plate, symbol Switch:SW_MEC_5G_LED
- removed SW53: L, Button_Switch_Keyboard:SW_Cherry_MX_1.00u_Plate, symbol Switch:SW_MEC_5G_LED
- removed SW54: 0, Button_Switch_Keyboard:SW_Cherry_MX_1.00u_Plate, symbol Switch:SW_MEC_5G_LED
- removed SW55: ., Button_Switch_Keyboard:SW_Cherry_MX_1.00u_Plate, symbol Switch:SW_MEC_5G_LED
- removed SW56: P, Button_Switch_Keyboard:SW_Cherry_MX_1.00u_Plate, symbol Switch:SW_MEC_5G_LED
- removed SW57: ;, Button_Switch_Keyboard:SW_Cherry_MX_1.00u_Plate, symbol Switch:SW_MEC_5G_LED
- removed SW58: F9, Button_Switch_Keyboard:SW_Cherry_MX_1.00u_Plate, symbol Switch:SW_MEC_5G_LED
- removed SW59: -, Button_Switch_Keyboard:SW_Cherry_MX_1.00u_Plate, symbol Switch:SW_MEC_5G_LED
- removed SW6, SW77: Ctrl, Button_Switch_Keyboard:SW_Cherry_MX_1.25u_Plate, symbol Switch:SW_MEC_5G_LED
- removed SW60: /, Button_Switch_Keyboard:SW_Cherry_MX_1.00u_Plate, symbol Switch:SW_MEC_5G_LED
- removed SW62: @, Button_Switch_Keyboard:SW_Cherry_MX_1.00u_Plate, symbol Switch:SW_MEC_5G_LED
- removed SW63: :, Button_Switch_Keyboard:SW_Cherry_MX_1.00u_Plate, symbol Switch:SW_MEC_5G_LED
- removed SW64: F10, Button_Switch_Keyboard:SW_Cherry_MX_1.00u_Plate, symbol Switch:SW_MEC_5G_LED
- removed SW65: ^, Button_Switch_Keyboard:SW_Cherry_MX_1.00u_Plate, symbol Switch:SW_MEC_5G_LED
- removed SW66, SW71: \\, Button_Switch_Keyboard:SW_Cherry_MX_1.00u_Plate, symbol Switch:SW_MEC_5G_LED
- removed SW68: [, Button_Switch_Keyboard:SW_Cherry_MX_1.00u_Plate, symbol Switch:SW_MEC_5G_LED
- removed SW69: ], Button_Switch_Keyboard:SW_Cherry_MX_1.00u_Plate, symbol Switch:SW_MEC_5G_LED
- removed SW7: F1, Button_Switch_Keyboard:SW_Cherry_MX_1.00u_Plate, symbol Switch:SW_MEC_5G_LED
- removed SW70: F11, Button_Switch_Keyboard:SW_Cherry_MX_1.00u_Plate, symbol Switch:SW_MEC_5G_LED
- removed SW72, SW9: Fn, Button_Switch_Keyboard:SW_Cherry_MX_1.25u_Plate, symbol Switch:SW_MEC_5G_LED
- removed SW73: F12, Button_Switch_Keyboard:SW_Cherry_MX_1.00u_Plate, symbol Switch:SW_MEC_5G_LED
- removed SW74: BS, Button_Switch_Keyboard:SW_Cherry_MX_1.00u_Plate, symbol Switch:SW_MEC_5G_LED
- removed SW75: Enter, Button_Switch_Keyboard:SW_Cherry_MX_ISOEnter_Plate, symbol Switch:SW_MEC_5G_LED
- removed SW76: Shift, Button_Switch_Keyboard:SW_Cherry_MX_1.75u_Plate, symbol Switch:SW_MEC_5G_LED
- removed SW78: PrtSc, Button_Switch_Keyboard:SW_Cherry_MX_1.00u_Plate, symbol Switch:SW_MEC_5G_LED
- removed SW79: Delete, Button_Switch_Keyboard:SW_Cherry_MX_1.00u_Plate, symbol Switch:SW_MEC_5G_LED
- removed SW8: 1, Button_Switch_Keyboard:SW_Cherry_MX_1.00u_Plate, symbol Switch:SW_MEC_5G_LED
- removed SW80: Left, Button_Switch_Keyboard:SW_Cherry_MX_1.00u_Plate, symbol Switch:SW_MEC_5G_LED
- removed SW81: Home, Button_Switch_Keyboard:SW_Cherry_MX_1.00u_Plate, symbol Switch:SW_MEC_5G_LED
- removed SW82: End, Button_Switch_Keyboard:SW_Cherry_MX_1.00u_Plate, symbol Switch:SW_MEC_5G_LED
- removed SW83: Up, Button_Switch_Keyboard:SW_Cherry_MX_1.00u_Plate, symbol Switch:SW_MEC_5G_LED
- removed SW84: Dn, Button_Switch_Keyboard:SW_Cherry_MX_1.00u_Plate, symbol Switch:SW_MEC_5G_LED
- removed SW85: PgUp, Button_Switch_Keyboard:SW_Cherry_MX_1.00u_Plate, symbol Switch:SW_MEC_5G_LED
- removed SW86: PgDn, Button_Switch_Keyboard:SW_Cherry_MX_1.00u_Plate, symbol Switch:SW_MEC_5G_LED
- removed SW87: Right, Button_Switch_Keyboard:SW_Cherry_MX_1.00u_Plate, symbol Switch:SW_MEC_5G_LED
- removed SW88: SW_MEC_5G, Button_Switch_THT:SW_PUSH_6mm_H5mm, symbol Switch:SW_MEC_5G
- removed U1: Master, Arduino:Sparkfun_Pro_Micro, symbol KiCAD-rescue:Sparkfun_Pro_Micro-Arduino
- removed U2: Slave, Arduino:Sparkfun_Pro_Micro, symbol KiCAD-rescue:Sparkfun_Pro_Micro-Arduino
- added D1, D10, D11, D12, D13, D14, D15, D16, D17, D18, D19, D2, D20, D21, D22, D23, D24, D25, D26, D27, D28, D29, D3, D30, D31, D32, D33, D34, D35, D36, D37, D38, D39, D4, D40, D41, D42, D43, D44, D45, D46, D47, D48, D49, D5, D50, D51, D52, D53, D54, D55, D56, D57, D58, D59, D6, D60, D61, D62, D63, D64, D65, D66, D67, D68, D69, D7, D70, D71, D72, D73, D74, D75, D76, D77, D78, D79, D8, D80, D81, D82, D83, D84, D85, D86, D87, D9: LED, LED_THT:LED_D3.0mm, symbol Device:LED
- added D100, D101, D102, D103, D104, D105, D106, D107, D108, D109, D110, D111, D112, D113, D114, D115, D116, D117, D118, D119, D120, D121, D122, D123, D124, D125, D126, D127, D128, D129, D130, D131, D132, D133, D134, D135, D136, D137, D138, D139, D140, D141, D142, D143, D144, D145, D146, D147, D148, D149, D150, D151, D152, D153, D154, D155, D156, D157, D158, D159, D160, D161, D162, D163, D164, D165, D166, D167, D168, D169, D170, D171, D172, D173, D174, D88, D89, D90, D91, D92, D93, D94, D95, D96, D97, D98, D99: 1N4148, LED_SMD:LED_0603_1608Metric, symbol Diode:1N4148
- added H1, H10, H11, H12, H13, H14, H15, H2, H3, H4, H5, H6, H7, H8, H9: MountingHole, MountingHole:MountingHole_3.5mm_Pad, symbol Mechanical:MountingHole
- added SW1, SW10, SW11, SW12, SW13, SW14, SW15, SW16, SW17, SW18, SW19, SW2, SW20, SW21, SW22, SW23, SW24, SW25, SW26, SW27, SW28, SW29, SW3, SW30, SW31, SW33, SW34, SW35, SW36, SW37, SW38, SW39, SW4, SW40, SW41, SW42, SW43, SW44, SW46, SW47, SW48, SW5, SW50, SW51, SW52, SW53, SW54, SW55, SW56, SW57, SW58, SW59, SW6, SW60, SW61, SW63, SW64, SW65, SW66, SW67, SW68, SW69, SW7, SW70, SW71, SW72, SW73, SW75, SW8, SW85, SW86, SW87, SW9: CherryMX, Button_Switch_Keyboard:SW_Cherry_MX_1.00u_PCB, symbol kicad_libraries:CherryMX
- added SW32, SW76, SW77, SW78, SW79, SW81, SW82, SW83, SW84: CherryMX, Button_Switch_Keyboard:SW_Cherry_MX_1.25u_PCB, symbol kicad_libraries:CherryMX
- added SW45: CherryMX, Button_Switch_Keyboard:SW_Cherry_MX_ISOEnter_PCB, symbol kicad_libraries:CherryMX
- added SW49: CherryMX, Button_Switch_Keyboard:SW_Cherry_MX_1.50u_PCB, symbol kicad_libraries:CherryMX
- added SW62, SW74: CherryMX, Button_Switch_Keyboard:SW_Cherry_MX_1.75u_PCB, symbol kicad_libraries:CherryMX
- added SW80: CherryMX, Button_Switch_Keyboard:SW_Cherry_MX_2.00u_PCB, symbol kicad_libraries:CherryMX
- added U1: Pico, RPi_Pico:RPi_Pico_SMD_TH, symbol RaspberryPi_Pico:Pico
- R1, R2, R3, R4, R5, R6: value 5k -> R
Connections:
- net labels added: Row6, Row7, Row8, Row9
- net labels removed: +5C, Col10, Col11, Col12, Col13, Col14, Col15, MasterRX, MasterTX, RST, VCC
- wire segments 875 -> 756
- no-connect marks 9 -> 14

Commit message: LED の点灯方法を変更。それぞれの LED に電流制限抵抗を追加。
Parts:
- added Q1: 2N7002, Package_TO_SOT_SMD:SOT-23, symbol Transistor_FET:2N7002
- added R10, R11, R12, R13, R14, R15, R16, R17, R18, R19, R20, R21, R22, R23, R24, R25, R26, R27, R28, R29, R30, R31, R32, R33, R34, R35, R36, R37, R38, R39, R40, R41, R42, R43, R44, R45, R46, R47, R48, R49, R50, R51, R52, R53, R54, R55, R56, R57, R58, R59, R60, R61, R62, R63, R64, R65, R66, R67, R68, R69, R7, R70, R71, R72, R73, R74, R75, R76, R77, R78, R79, R8, R80, R81, R82, R83, R84, R85, R86, R87, R9: 630, Resistor_SMD:R_0603_1608Metric, symbol Device:R
- added R88: 1k, Resistor_SMD:R_0603_1608Metric, symbol Device:R
- R1, R2, R3, R4, R5, R6: value R -> 630
- SW1, SW10, SW11, SW12, SW13, SW14, SW15, SW16, SW17, SW18, SW19, SW2, SW20, SW21, SW22, SW23, SW24, SW25, SW26, SW27, SW28, SW29, SW3, SW30, SW31, SW32, SW33, SW34, SW35, SW36, SW37, SW38, SW39, SW4, SW40, SW41, SW42, SW43, SW44, SW45, SW46, SW47, SW48, SW49, SW5, SW50, SW51, SW52, SW53, SW54, SW55, SW56, SW57, SW58, SW59, SW6, SW60, SW61, SW62, SW63, SW64, SW65, SW66, SW67, SW68, SW69, SW7, SW70, SW71, SW72, SW73, SW74, SW75, SW76, SW77, SW78, SW79, SW8, SW80, SW81, SW82, SW83, SW84, SW85, SW86, SW87, SW9: symbol kicad_libraries:CherryMX -> KiCAD-rescue:CherryMX-kicad_libraries
Connections:
- net Col1: now also U1.9 (GPIO6); no longer U1.7 (GPIO5)
- net Col4: now also U1.14 (GPIO10); no longer U1.12 (GPIO9)
- net Col5: now also U1.12 (GPIO9); no longer U1.11 (GPIO8)
- net Col6: now also U1.11 (GPIO8); no longer U1.10 (GPIO7)
- net Col7: now also U1.10 (GPIO7); no longer U1.9 (GPIO6)
- net Col8: now also U1.7 (GPIO5); no longer U1.6 (GPIO4)
- net Col9: now also U1.6 (GPIO4); no longer U1.5 (GPIO3)
- net GND: now also Q1.2 (S); no longer D1.1 (K), D10.1 (K), D11.1 (K), D12.1 (K), D13.1 (K), D14.1 (K), D15.1 (K), D16.1 (K), D17.1 (K), D18.1 (K), D19.1 (K), D2.1 (K), D20.1 (K), D21.1 (K), D22.1 (K), D23.1 (K), D24.1 (K), D25.1 (K), D26.1 (K), D27.1 (K), D28.1 (K), D29.1 (K), D3.1 (K), D30.1 (K), D31.1 (K), D32.1 (K), D33.1 (K), D34.1 (K), D35.1 (K), D36.1 (K), D37.1 (K), D38.1 (K), D39.1 (K), D4.1 (K), D40.1 (K), D41.1 (K), D42.1 (K), D43.1 (K), D44.1 (K), D45.1 (K), D46.1 (K), D47.1 (K), D48.1 (K), D49.1 (K), D5.1 (K), D50.1 (K), D51.1 (K), D52.1 (K), D53.1 (K), D54.1 (K), D55.1 (K), D56.1 (K), D57.1 (K), D58.1 (K), D59.1 (K), D6.1 (K), D60.1 (K), D61.1 (K), D62.1 (K), D63.1 (K), D64.1 (K), D65.1 (K), D66.1 (K), D67.1 (K), D68.1 (K), D69.1 (K), D7.1 (K), D70.1 (K), D71.1 (K), D72.1 (K), D73.1 (K), D74.1 (K), D75.1 (K), D76.1 (K), D77.1 (K), D78.1 (K), D79.1 (K), D8.1 (K), D80.1 (K), D81.1 (K), D82.1 (K), D83.1 (K), D84.1 (K), D85.1 (K), D86.1 (K), D87.1 (K), D9.1 (K)
- net PWM: now also R88.2; no longer R1.1, R2.1, R3.1, R4.1, R5.1, R6.1
- net Row0: now also U1.5 (GPIO3); no longer U1.14 (GPIO10)
- net VBUS: now reaches U1.40 (VBUS)
- net VBUS: now also R1.2, R2.2, R3.2, R4.2, R5.2, R6.2, R10.2, R11.2, R12.2, R13.2, R14.2, R15.2, R16.2, R17.2, R18.2, R19.2, R20.2, R21.2, R22.2, R23.2, R24.2, R25.2, R26.2, R27.2, R28.2, R29.2, R30.2, R31.2, R32.2, R33.2, R34.2, R35.2, R36.2, R37.2, R38.2, R39.2, R40.2, R41.2, R42.2, R43.2, R44.2, R45.2, R46.2, R47.2, R48.2, R49.2, R50.2, R51.2, R52.2, R53.2, R54.2, R55.2, R56.2, R57.2, R58.2, R59.2, R60.2, R61.2, R62.2, R63.2, R64.2, R65.2, R66.2, R67.2, R68.2, R69.2, R7.2, R70.2, R71.2, R72.2, R73.2, R74.2, R75.2, R76.2, R77.2, R78.2, R79.2, R8.2, R80.2, R81.2, R82.2, R83.2, R84.2, R85.2, R86.2, R87.2, R9.2
- new net: D1.2 (A), R1.1
- new net: D2.2 (A), R2.1
- new net: D3.2 (A), R3.1
- new net: D4.2 (A), R4.1
- new net: D5.2 (A), R5.1
- new net: Q1.1 (G), R88.1
- new net: D6.2 (A), R6.1
- new net: D7.2 (A), R7.1
- new net: D8.2 (A), R8.1
- new net: D9.2 (A), R9.1
- new net: D10.2 (A), R10.1
- new net: D11.2 (A), R11.1
- new net: D12.2 (A), R12.1
- new net: D13.2 (A), R13.1
- new net: D14.2 (A), R14.1
- new net: D15.2 (A), R15.1
- new net: D16.2 (A), R16.1
- new net: D17.2 (A), R17.1
- new net: D18.2 (A), R18.1
- new net: D19.2 (A), R19.1
- new net: D20.2 (A), R20.1
- new net: D21.2 (A), R21.1
- new net: D22.2 (A), R22.1
- new net: D23.2 (A), R23.1
- new net: D24.2 (A), R24.1
- new net: D25.2 (A), R25.1
- new net: D26.2 (A), R26.1
- new net: D27.2 (A), R27.1
- new net: D28.2 (A), R28.1
- new net: D29.2 (A), R29.1
- new net: D30.2 (A), R30.1
- new net: D31.2 (A), R31.1
- new net: D32.2 (A), R32.1
- new net: D33.2 (A), R33.1
- new net: D34.2 (A), R34.1
- new net: D35.2 (A), R35.1
- new net: D36.2 (A), R36.1
- new net: D37.2 (A), R37.1
- new net: D38.2 (A), R38.1
- new net: D39.2 (A), R39.1
- new net: D40.2 (A), R40.1
- new net: D41.2 (A), R41.1
- new net: D42.2 (A), R42.1
- new net: D43.2 (A), R43.1
- new net: D1.1 (K), D10.1 (K), D11.1 (K), D12.1 (K), D13.1 (K), D14.1 (K), D15.1 (K), D16.1 (K), D17.1 (K), D18.1 (K), D19.1 (K), D2.1 (K), D20.1 (K), D21.1 (K), D22.1 (K), D23.1 (K), D24.1 (K), D25.1 (K), D26.1 (K), D27.1 (K), D28.1 (K), D29.1 (K), D3.1 (K), D30.1 (K), D31.1 (K), D32.1 (K), D33.1 (K), D34.1 (K), D35.1 (K), D36.1 (K), D37.1 (K), D38.1 (K), D39.1 (K), D4.1 (K), D40.1 (K), D41.1 (K), D42.1 (K), D43.1 (K), D44.1 (K), D45.1 (K), D46.1 (K), D47.1 (K), D48.1 (K), D49.1 (K), D5.1 (K), D50.1 (K), D51.1 (K), D52.1 (K), D53.1 (K), D54.1 (K), D55.1 (K), D56.1 (K), D57.1 (K), D58.1 (K), D59.1 (K), D6.1 (K), D60.1 (K), D61.1 (K), D62.1 (K), D63.1 (K), D64.1 (K), D65.1 (K), D66.1 (K), D67.1 (K), D68.1 (K), D69.1 (K), D7.1 (K), D70.1 (K), D71.1 (K), D72.1 (K), D73.1 (K), D74.1 (K), D75.1 (K), D76.1 (K), D77.1 (K), D78.1 (K), D79.1 (K), D8.1 (K), D80.1 (K), D81.1 (K), D82.1 (K), D83.1 (K), D84.1 (K), D85.1 (K), D86.1 (K), D87.1 (K), D9.1 (K), Q1.3 (D)
- new net: D60.2 (A), R60.1
- new net: D61.2 (A), R61.1
- new net: D62.2 (A), R62.1
- new net: D63.2 (A), R63.1
- new net: D64.2 (A), R64.1
- new net: D65.2 (A), R65.1
- new net: D66.2 (A), R66.1
- new net: D67.2 (A), R67.1
- new net: D68.2 (A), R68.1
- new net: D69.2 (A), R69.1
- new net: D70.2 (A), R70.1
- new net: D71.2 (A), R71.1
- new net: D72.2 (A), R72.1
- new net: D73.2 (A), R73.1
- new net: D74.2 (A), R74.1
- new net: D75.2 (A), R75.1
- new net: D76.2 (A), R76.1
- new net: D77.2 (A), R77.1
- new net: D78.2 (A), R78.1
- new net: D79.2 (A), R79.1
- new net: D80.2 (A), R80.1
- new net: D81.2 (A), R81.1
- new net: D82.2 (A), R82.1
- new net: D83.2 (A), R83.1
- new net: D84.2 (A), R84.1
- new net: D85.2 (A), R85.1
- new net: D86.2 (A), R86.1
- new net: D87.2 (A), R87.1
- new net: D44.2 (A), R44.1
- new net: D45.2 (A), R45.1
- new net: D46.2 (A), R46.1
- new net: D47.2 (A), R47.1
- new net: D48.2 (A), R48.1
- new net: D49.2 (A), R49.1
- new net: D50.2 (A), R50.1
- new net: D51.2 (A), R51.1
- new net: D52.2 (A), R52.1
- new net: D53.2 (A), R53.1
- new net: D54.2 (A), R54.1
- new net: D55.2 (A), R55.1
- new net: D56.2 (A), R56.1
- new net: D57.2 (A), R57.1
- new net: D58.2 (A), R58.1
- new net: D59.2 (A), R59.1
- no-connect marks 14 -> 13
Other:
- moved on the sheet: D1, D10, D100, D101, D102, D103, D104, D105, D106, D107, D108, D109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
