File: pcb/main/_autosave-KiCAD.sch (KiCad schematic (older format))
At the start: 368 parts, among them Q1 2N7002, SW1 CherryMX, SW10 CherryMX, SW11 CherryMX, SW12 CherryMX, SW13 CherryMX, SW14 CherryMX, SW15 CherryMX, SW16 CherryMX, SW17 CherryMX, SW18 CherryMX, SW19 CherryMX, SW2 CherryMX, SW20 CherryMX, SW21 CherryMX, SW22 CherryMX, SW23 CherryMX, SW24 CherryMX, SW25 CherryMX, SW26 CherryMX, SW27 CherryMX, SW28 CherryMX, SW29 CherryMX, SW3 CherryMX, SW30 CherryMX, SW31 CherryMX, SW32 CherryMX, SW33 CherryMX, SW34 CherryMX, SW35 CherryMX, SW36 CherryMX, SW37 CherryMX, SW38 CherryMX, SW39 CherryMX, SW4 CherryMX, SW40 CherryMX, SW41 CherryMX, SW42 CherryMX, SW43 CherryMX, SW44 CherryMX, SW45 CherryMX, SW46 CherryMX, SW47 CherryMX, SW48 CherryMX, SW49 CherryMX, SW5 CherryMX, SW50 CherryMX, SW51 CherryMX, SW52 CherryMX, SW53 CherryMX, SW54 CherryMX, SW55 CherryMX, SW56 CherryMX, SW57 CherryMX, SW58 CherryMX, SW59 CherryMX, SW6 CherryMX, SW60 CherryMX, SW61 CherryMX, SW62 CherryMX, SW63 CherryMX, SW64 CherryMX, SW65 CherryMX, SW66 CherryMX, SW67 CherryMX, SW68 CherryMX, SW69 CherryMX, SW7 CherryMX, SW70 CherryMX, SW71 CherryMX, SW72 CherryMX, SW73 CherryMX, SW74 CherryMX, SW75 CherryMX, SW76 CherryMX, SW77 CherryMX, SW78 CherryMX, SW79 CherryMX, SW8 CherryMX, SW80 CherryMX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

Commit message: GS間抵抗を追加。G抵抗を追加。なんかスイッチのフットプリント一つ消えちゃった
Parts:
- C1: footprint (none) -> Capacitor_SMD:C_0603_1608Metric
- R89: footprint (none) -> Resistor_SMD:R_0603_1608Metric
Changed lines of the file:
@@
 F 0 "C1" H 3565 7046 50  0000 L CNN
 F 1 "3.3u" H 3565 6955 50  0000 L CNN
-F 2 "" H 3488 6850 50  0001 C CNN
+F 2 "Capacitor_SMD:C_0603_1608Metric" H 3488 6850 50  0001 C CNN
 F 3 "~" H 3450 7000 50  0001 C CNN
 	1    3450 7000
@@
 F 0 "R89" H 2120 5296 50  0000 L CNN
 F 1 "10k" H 2120 5205 50  0000 L CNN
-F 2 "" V 1980 5250 50  0001 C CNN
+F 2 "Resistor_SMD:R_0603_1608Metric" V 1980 5250 50  0001 C CNN
 F 3 "~" H 2050 5250 50  0001 C CNN
 	1    2050 5250
