File: pcb/main/KiCAD.kicad_pcb (KiCad board)
At the start: 2 copper layers, 365.8 x 137.2 mm, 283 parts, among them SW1 CherryMX, SW10 CherryMX, SW11 CherryMX, SW12 CherryMX, SW13 CherryMX, SW14 CherryMX, SW15 CherryMX, SW16 CherryMX, SW17 CherryMX, SW18 CherryMX, SW19 CherryMX, SW2 CherryMX, SW20 CherryMX, SW21 CherryMX, SW22 CherryMX, SW23 CherryMX, SW24 CherryMX, SW25 CherryMX, SW26 CherryMX, SW27 CherryMX, SW28 CherryMX, SW29 CherryMX, SW3 CherryMX, SW30 CherryMX, SW31 CherryMX, SW32 CherryMX, SW33 CherryMX, SW34 CherryMX, SW35 CherryMX, SW36 CherryMX, SW37 CherryMX, SW38 CherryMX, SW39 CherryMX, SW4 CherryMX, SW40 CherryMX, SW41 CherryMX, SW42 CherryMX, SW43 CherryMX, SW44 CherryMX, SW45 CherryMX, SW46 CherryMX, SW47 CherryMX, SW48 CherryMX, SW49 CherryMX, SW5 CherryMX, SW50 CherryMX, SW51 CherryMX, SW52 CherryMX, SW53 CherryMX, SW54 CherryMX, SW55 CherryMX, SW56 CherryMX, SW57 CherryMX, SW58 CherryMX, SW59 CherryMX, SW6 CherryMX, SW60 CherryMX, SW61 CherryMX, SW62 CherryMX, SW63 CherryMX, SW64 CherryMX, SW65 CherryMX, SW66 CherryMX, SW67 CherryMX, SW68 CherryMX, SW69 CherryMX, SW7 CherryMX, SW70 CherryMX, SW71 CherryMX, SW72 CherryMX, SW73 CherryMX, SW74 CherryMX, SW75 CherryMX, SW76 CherryMX, SW77 CherryMX, SW78 CherryMX, SW79 CherryMX, SW8 CherryMX, SW80 CherryMX, SW81 CherryMX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

Commit message: LED の点灯方法を変更。それぞれの LED に電流制限抵抗を追加。
Parts:
- added Q1: 2N7002, Package_TO_SOT_SMD:SOT-23, B.Cu at (148.0, 93.3)
- added R10: 630, Resistor_SMD:R_0603_1608Metric, B.Cu at (261.6, 67.9)
- added R11: 630, Resistor_SMD:R_0603_1608Metric, B.Cu at (280.7, 67.9)
- added R12: 630, Resistor_SMD:R_0603_1608Metric, B.Cu at (299.7, 67.9)
- added R13: 630, Resistor_SMD:R_0603_1608Metric, B.Cu at (318.8, 67.9)
- added R14: 630, Resistor_SMD:R_0603_1608Metric, B.Cu at (52.1, 96.5)
- added R15: 630, Resistor_SMD:R_0603_1608Metric, B.Cu at (71.1, 96.5)
- added R16: 630, Resistor_SMD:R_0603_1608Metric, B.Cu at (90.2, 96.5)
- added R17: 630, Resistor_SMD:R_0603_1608Metric, B.Cu at (109.2, 96.5)
- added R18: 630, Resistor_SMD:R_0603_1608Metric, B.Cu at (128.3, 96.5)
- added R19: 630, Resistor_SMD:R_0603_1608Metric, B.Cu at (149.9, 96.5)
- added R20: 630, Resistor_SMD:R_0603_1608Metric, B.Cu at (166.4, 96.5)
- added R21: 630, Resistor_SMD:R_0603_1608Metric, B.Cu at (185.4, 96.5)
- added R22: 630, Resistor_SMD:R_0603_1608Metric, B.Cu at (204.5, 96.5)
- added R23: 630, Resistor_SMD:R_0603_1608Metric, B.Cu at (223.5, 96.5)
- added R24: 630, Resistor_SMD:R_0603_1608Metric, B.Cu at (242.6, 96.5)
- added R25: 630, Resistor_SMD:R_0603_1608Metric, B.Cu at (261.6, 96.5)
- added R26: 630, Resistor_SMD:R_0603_1608Metric, B.Cu at (280.7, 96.5)
- added R27: 630, Resistor_SMD:R_0603_1608Metric, B.Cu at (299.7, 96.5)
- added R28: 630, Resistor_SMD:R_0603_1608Metric, B.Cu at (318.8, 96.5)
- added R29: 630, Resistor_SMD:R_0603_1608Metric, B.Cu at (347.3, 96.5)
- added R30: 630, Resistor_SMD:R_0603_1608Metric, B.Cu at (366.4, 96.5)
- added R31: 630, Resistor_SMD:R_0603_1608Metric, B.Cu at (385.4, 96.5)
- added R32: 630, Resistor_SMD:R_0603_1608Metric, B.Cu at (56.5, 115.6)
- added R33: 630, Resistor_SMD:R_0603_1608Metric, B.Cu at (80.6, 115.6)
- added R34: 630, Resistor_SMD:R_0603_1608Metric, B.Cu at (99.1, 115.6)
- added R35: 630, Resistor_SMD:R_0603_1608Metric, B.Cu at (119.4, 115.6)
- added R36: 630, Resistor_SMD:R_0603_1608Metric, B.Cu at (137.8, 115.6)
- added R37: 630, Resistor_SMD:R_0603_1608Metric, B.Cu at (156.8, 115.6)
- added R38: 630, Resistor_SMD:R_0603_1608Metric, B.Cu at (176.5, 115.6)
- added R39: 630, Resistor_SMD:R_0603_1608Metric, B.Cu at (194.9, 115.6)
- added R40: 630, Resistor_SMD:R_0603_1608Metric, B.Cu at (214.0, 115.6)
- added R41: 630, Resistor_SMD:R_0603_1608Metric, B.Cu at (233.0, 115.6)
- added R42: 630, Resistor_SMD:R_0603_1608Metric, B.Cu at (252.1, 115.6)
- added R43: 630, Resistor_SMD:R_0603_1608Metric, B.Cu at (271.1, 115.6)
- added R44: 630, Resistor_SMD:R_0603_1608Metric, B.Cu at (290.2, 115.6)
- added R45: 630, Resistor_SMD:R_0603_1608Metric, B.Cu at (316.2, 124.9)
- added R46: 630, Resistor_SMD:R_0603_1608Metric, B.Cu at (347.3, 115.6)
- added R47: 630, Resistor_SMD:R_0603_1608Metric, B.Cu at (366.4, 115.6)
- added R48: 630, Resistor_SMD:R_0603_1608Metric, B.Cu at (385.4, 115.6)
- added R49: 630, Resistor_SMD:R_0603_1608Metric, B.Cu at (59.7, 134.6)
- added R50: 630, Resistor_SMD:R_0603_1608Metric, B.Cu at (85.1, 134.6)
- added R51: 630, Resistor_SMD:R_0603_1608Metric, B.Cu at (104.8, 134.6)
- added R52: 630, Resistor_SMD:R_0603_1608Metric, B.Cu at (123.2, 134.6)
- added R53: 630, Resistor_SMD:R_0603_1608Metric, B.Cu at (142.2, 134.6)
- added R54: 630, Resistor_SMD:R_0603_1608Metric, B.Cu at (161.9, 134.6)
- added R55: 630, Resistor_SMD:R_0603_1608Metric, B.Cu at (181.0, 134.6)
- added R56: 630, Resistor_SMD:R_0603_1608Metric, B.Cu at (200.0, 134.6)
- added R57: 630, Resistor_SMD:R_0603_1608Metric, B.Cu at (219.1, 134.6)
- added R58: 630, Resistor_SMD:R_0603_1608Metric, B.Cu at (238.1, 134.6)
- added R59: 630, Resistor_SMD:R_0603_1608Metric, B.Cu at (256.5, 134.6)
- added R60: 630, Resistor_SMD:R_0603_1608Metric, B.Cu at (276.2, 134.6)
- added R61: 630, Resistor_SMD:R_0603_1608Metric, B.Cu at (288.9, 134.6)
- added R62: 630, Resistor_SMD:R_0603_1608Metric, B.Cu at (62.2, 153.7)
- added R63: 630, Resistor_SMD:R_0603_1608Metric, B.Cu at (90.2, 153.7)
- added R64: 630, Resistor_SMD:R_0603_1608Metric, B.Cu at (109.2, 153.7)
- added R65: 630, Resistor_SMD:R_0603_1608Metric, B.Cu at (128.3, 153.7)
- added R66: 630, Resistor_SMD:R_0603_1608Metric, B.Cu at (147.3, 153.7)
- added R67: 630, Resistor_SMD:R_0603_1608Metric, B.Cu at (166.4, 153.7)
- added R68: 630, Resistor_SMD:R_0603_1608Metric, B.Cu at (185.4, 153.7)
- added R69: 630, Resistor_SMD:R_0603_1608Metric, B.Cu at (204.5, 153.7)
- added R7: 630, Resistor_SMD:R_0603_1608Metric, B.Cu at (194.9, 67.9)
- added R70: 630, Resistor_SMD:R_0603_1608Metric, B.Cu at (223.5, 153.7)
- added R71: 630, Resistor_SMD:R_0603_1608Metric, B.Cu at (242.6, 153.7)
- added R72: 630, Resistor_SMD:R_0603_1608Metric, B.Cu at (261.6, 153.7)
- added R73: 630, Resistor_SMD:R_0603_1608Metric, B.Cu at (280.7, 153.7)
- added R74: 630, Resistor_SMD:R_0603_1608Metric, B.Cu at (309.2, 153.7)
- added R75: 630, Resistor_SMD:R_0603_1608Metric, B.Cu at (366.4, 153.7)
- added R76: 630, Resistor_SMD:R_0603_1608Metric, B.Cu at (54.6, 172.7)
- added R77: 630, Resistor_SMD:R_0603_1608Metric, B.Cu at (78.7, 172.7)
- added R78: 630, Resistor_SMD:R_0603_1608Metric, B.Cu at (101.6, 172.7)
- added R79: 630, Resistor_SMD:R_0603_1608Metric, B.Cu at (125.7, 172.7)
- added R8: 630, Resistor_SMD:R_0603_1608Metric, B.Cu at (214.0, 67.9)
- added R80: 630, Resistor_SMD:R_0603_1608Metric, B.Cu at (185.4, 172.7)
- added R81: 630, Resistor_SMD:R_0603_1608Metric, B.Cu at (245.1, 172.7)
- added R82: 630, Resistor_SMD:R_0603_1608Metric, B.Cu at (269.2, 172.7)
- added R83: 630, Resistor_SMD:R_0603_1608Metric, B.Cu at (292.1, 172.7)
- added R84: 630, Resistor_SMD:R_0603_1608Metric, B.Cu at (316.2, 172.7)
- added R85: 630, Resistor_SMD:R_0603_1608Metric, B.Cu at (347.3, 172.7)
- added R86: 630, Resistor_SMD:R_0603_1608Metric, B.Cu at (366.4, 172.7)
- added R87: 630, Resistor_SMD:R_0603_1608Metric, B.Cu at (386.1, 172.7)
- added R88: 1k, Resistor_SMD:R_0603_1608Metric, B.Cu at (143.5, 92.1)
- added R9: 630, Resistor_SMD:R_0603_1608Metric, B.Cu at (233.0, 67.9)
- R1, R2, R3, R4, R5, R6: value R -> 630
- moved R6 142.6 mm to (182.2, 67.9), turned to 90 degrees
- moved R5 106.4 mm to (147.3, 67.9), turned to 90 degrees
- moved R4 82.2 mm to (128.3, 67.9), turned to 90 degrees
- moved R1 66.8 mm to (52.1, 67.9), turned to 90 degrees
- moved R2 63.1 mm to (90.2, 67.9), turned to 90 degrees
- moved R3 54.5 mm to (109.2, 67.9), turned to 90 degrees
- moved D92 7.62 mm to (149.9, 74.9), turned to 270 degrees
- moved H13 6.35 mm to (171.4, 64.8)
- moved H7 6.35 mm to (120.7, 64.8)
- moved D163 4.96 mm to (61.0, 183.5), turned to 180 degrees
- moved D164 4.49 mm to (84.5, 183.5), turned to 180 degrees
- moved D165 4.49 mm to (108.6, 183.5), turned to 180 degrees
- moved D166 4.07 mm to (132.1, 183.5), turned to 180 degrees
Connections:
- D1 pad 1: GND -> Net-(D1-Pad1)
- D10 pad 1: GND -> Net-(D1-Pad1)
- D10 pad 2: Net-(D1-Pad2) -> Net-(D10-Pad2)
- D11 pad 1: GND -> Net-(D1-Pad1)
- D11 pad 2: Net-(D1-Pad2) -> Net-(D11-Pad2)
- D12 pad 1: GND -> Net-(D1-Pad1)
- D12 pad 2: Net-(D1-Pad2) -> Net-(D12-Pad2)
- D13 pad 1: GND -> Net-(D1-Pad1)
- D13 pad 2: Net-(D1-Pad2) -> Net-(D13-Pad2)
- D14 pad 1: GND -> Net-(D1-Pad1)
- D14 pad 2: Net-(D1-Pad2) -> Net-(D14-Pad2)
- D15 pad 1: GND -> Net-(D1-Pad1)
- D15 pad 2: Net-(D1-Pad2) -> Net-(D15-Pad2)
- D16 pad 1: GND -> Net-(D1-Pad1)
- D17 pad 1: GND -> Net-(D1-Pad1)
- D17 pad 2: Net-(D16-Pad2) -> Net-(D17-Pad2)
- D18 pad 1: GND -> Net-(D1-Pad1)
- D18 pad 2: Net-(D16-Pad2) -> Net-(D18-Pad2)
- D19 pad 1: GND -> Net-(D1-Pad1)
- D19 pad 2: Net-(D16-Pad2) -> Net-(D19-Pad2)
- D2 pad 1: GND -> Net-(D1-Pad1)
- D2 pad 2: Net-(D1-Pad2) -> Net-(D2-Pad2)
- D20 pad 1: GND -> Net-(D1-Pad1)
- D20 pad 2: Net-(D16-Pad2) -> Net-(D20-Pad2)
- D21 pad 1: GND -> Net-(D1-Pad1)
- D21 pad 2: Net-(D16-Pad2) -> Net-(D21-Pad2)
- D22 pad 1: GND -> Net-(D1-Pad1)
- D22 pad 2: Net-(D16-Pad2) -> Net-(D22-Pad2)
- D23 pad 1: GND -> Net-(D1-Pad1)
- D23 pad 2: Net-(D16-Pad2) -> Net-(D23-Pad2)
- D24 pad 1: GND -> Net-(D1-Pad1)
- D24 pad 2: Net-(D16-Pad2) -> Net-(D24-Pad2)
- D25 pad 1: GND -> Net-(D1-Pad1)
- D25 pad 2: Net-(D16-Pad2) -> Net-(D25-Pad2)
- D26 pad 1: GND -> Net-(D1-Pad1)
- D26 pad 2: Net-(D16-Pad2) -> Net-(D26-Pad2)
- D27 pad 1: GND -> Net-(D1-Pad1)
- D27 pad 2: Net-(D16-Pad2) -> Net-(D27-Pad2)
- D28 pad 1: GND -> Net-(D1-Pad1)
- D28 pad 2: Net-(D16-Pad2) -> Net-(D28-Pad2)
- D29 pad 1: GND -> Net-(D1-Pad1)
- D29 pad 2: Net-(D16-Pad2) -> Net-(D29-Pad2)
- D3 pad 1: GND -> Net-(D1-Pad1)
- D3 pad 2: Net-(D1-Pad2) -> Net-(D3-Pad2)
- D30 pad 1: GND -> Net-(D1-Pad1)
- D30 pad 2: Net-(D16-Pad2) -> Net-(D30-Pad2)
- D31 pad 1: GND -> Net-(D1-Pad1)
- D32 pad 1: GND -> Net-(D1-Pad1)
- D32 pad 2: Net-(D31-Pad2) -> Net-(D32-Pad2)
- D33 pad 1: GND -> Net-(D1-Pad1)
- D33 pad 2: Net-(D31-Pad2) -> Net-(D33-Pad2)
- D34 pad 1: GND -> Net-(D1-Pad1)
- D34 pad 2: Net-(D31-Pad2) -> Net-(D34-Pad2)
- D35 pad 1: GND -> Net-(D1-Pad1)
- D35 pad 2: Net-(D31-Pad2) -> Net-(D35-Pad2)
- D36 pad 1: GND -> Net-(D1-Pad1)
- D36 pad 2: Net-(D31-Pad2) -> Net-(D36-Pad2)
- D37 pad 1: GND -> Net-(D1-Pad1)
- D37 pad 2: Net-(D31-Pad2) -> Net-(D37-Pad2)
- D38 pad 1: GND -> Net-(D1-Pad1)
- D38 pad 2: Net-(D31-Pad2) -> Net-(D38-Pad2)
- D39 pad 1: GND -> Net-(D1-Pad1)
- D39 pad 2: Net-(D31-Pad2) -> Net-(D39-Pad2)
- D4 pad 1: GND -> Net-(D1-Pad1)
- D4 pad 2: Net-(D1-Pad2) -> Net-(D4-Pad2)
- D40 pad 1: GND -> Net-(D1-Pad1)
- D40 pad 2: Net-(D31-Pad2) -> Net-(D40-Pad2)
- D41 pad 1: GND -> Net-(D1-Pad1)
- D41 pad 2: Net-(D31-Pad2) -> Net-(D41-Pad2)
- D42 pad 1: GND -> Net-(D1-Pad1)
- D42 pad 2: Net-(D31-Pad2) -> Net-(D42-Pad2)
- D43 pad 1: GND -> Net-(D1-Pad1)
- D43 pad 2: Net-(D31-Pad2) -> Net-(D43-Pad2)
- D44 pad 1: GND -> Net-(D1-Pad1)
- D44 pad 2: Net-(D31-Pad2) -> Net-(D44-Pad2)
- D45 pad 1: GND -> Net-(D1-Pad1)
- D45 pad 2: Net-(D31-Pad2) -> Net-(D45-Pad2)
- D46 pad 1: GND -> Net-(D1-Pad1)
- D47 pad 1: GND -> Net-(D1-Pad1)
- D47 pad 2: Net-(D46-Pad2) -> Net-(D47-Pad2)
- D48 pad 1: GND -> Net-(D1-Pad1)
- D48 pad 2: Net-(D46-Pad2) -> Net-(D48-Pad2)
- D49 pad 1: GND -> Net-(D1-Pad1)
- D49 pad 2: Net-(D46-Pad2) -> Net-(D49-Pad2)
- D5 pad 1: GND -> Net-(D1-Pad1)
- D5 pad 2: Net-(D1-Pad2) -> Net-(D5-Pad2)
- D50 pad 1: GND -> Net-(D1-Pad1)
- D50 pad 2: Net-(D46-Pad2) -> Net-(D50-Pad2)
- D51 pad 1: GND -> Net-(D1-Pad1)
- D51 pad 2: Net-(D46-Pad2) -> Net-(D51-Pad2)
- D52 pad 1: GND -> Net-(D1-Pad1)
- D52 pad 2: Net-(D46-Pad2) -> Net-(D52-Pad2)
- D53 pad 1: GND -> Net-(D1-Pad1)
- D53 pad 2: Net-(D46-Pad2) -> Net-(D53-Pad2)
- D54 pad 1: GND -> Net-(D1-Pad1)
- D54 pad 2: Net-(D46-Pad2) -> Net-(D54-Pad2)
- D55 pad 1: GND -> Net-(D1-Pad1)
- D55 pad 2: Net-(D46-Pad2) -> Net-(D55-Pad2)
- D56 pad 1: GND -> Net-(D1-Pad1)
- D56 pad 2: Net-(D46-Pad2) -> Net-(D56-Pad2)
- D57 pad 1: GND -> Net-(D1-Pad1)
- D57 pad 2: Net-(D46-Pad2) -> Net-(D57-Pad2)
- D58 pad 1: GND -> Net-(D1-Pad1)
- D58 pad 2: Net-(D46-Pad2) -> Net-(D58-Pad2)
- D59 pad 1: GND -> Net-(D1-Pad1)
- D59 pad 2: Net-(D46-Pad2) -> Net-(D59-Pad2)
- D6 pad 1: GND -> Net-(D1-Pad1)
- D6 pad 2: Net-(D1-Pad2) -> Net-(D6-Pad2)
- D60 pad 1: GND -> Net-(D1-Pad1)
- D61 pad 1: GND -> Net-(D1-Pad1)
- D61 pad 2: Net-(D60-Pad2) -> Net-(D61-Pad2)
- D62 pad 1: GND -> Net-(D1-Pad1)
- D62 pad 2: Net-(D60-Pad2) -> Net-(D62-Pad2)
- D63 pad 1: GND -> Net-(D1-Pad1)
- D63 pad 2: Net-(D60-Pad2) -> Net-(D63-Pad2)
- D64 pad 1: GND -> Net-(D1-Pad1)
- D64 pad 2: Net-(D60-Pad2) -> Net-(D64-Pad2)
- D65 pad 1: GND -> Net-(D1-Pad1)
- D65 pad 2: Net-(D60-Pad2) -> Net-(D65-Pad2)
- D66 pad 1: GND -> Net-(D1-Pad1)
- D66 pad 2: Net-(D60-Pad2) -> Net-(D66-Pad2)
- D67 pad 1: GND -> Net-(D1-Pad1)
- D67 pad 2: Net-(D60-Pad2) -> Net-(D67-Pad2)
- D68 pad 1: GND -> Net-(D1-Pad1)
- D68 pad 2: Net-(D60-Pad2) -> Net-(D68-Pad2)
- D69 pad 1: GND -> Net-(D1-Pad1)
- D69 pad 2: Net-(D60-Pad2) -> Net-(D69-Pad2)
- D7 pad 1: GND -> Net-(D1-Pad1)
- D7 pad 2: Net-(D1-Pad2) -> Net-(D7-Pad2)
- D70 pad 1: GND -> Net-(D1-Pad1)
- D70 pad 2: Net-(D60-Pad2) -> Net-(D70-Pad2)
- D71 pad 1: GND -> Net-(D1-Pad1)
- D71 pad 2: Net-(D60-Pad2) -> Net-(D71-Pad2)
- D72 pad 1: GND -> Net-(D1-Pad1)
- D72 pad 2: Net-(D60-Pad2) -> Net-(D72-Pad2)
- D73 pad 1: GND -> Net-(D1-Pad1)
- D73 pad 2: Net-(D60-Pad2) -> Net-(D73-Pad2)
- D74 pad 1: GND -> Net-(D1-Pad1)
- D75 pad 1: GND -> Net-(D1-Pad1)
- D75 pad 2: Net-(D74-Pad2) -> Net-(D75-Pad2)
- D76 pad 1: GND -> Net-(D1-Pad1)
- D76 pad 2: Net-(D74-Pad2) -> Net-(D76-Pad2)
- D77 pad 1: GND -> Net-(D1-Pad1)
- D77 pad 2: Net-(D74-Pad2) -> Net-(D77-Pad2)
- D78 pad 1: GND -> Net-(D1-Pad1)
- D78 pad 2: Net-(D74-Pad2) -> Net-(D78-Pad2)
- D79 pad 1: GND -> Net-(D1-Pad1)
- D79 pad 2: Net-(D74-Pad2) -> Net-(D79-Pad2)
- D8 pad 1: GND -> Net-(D1-Pad1)
- D8 pad 2: Net-(D1-Pad2) -> Net-(D8-Pad2)
- D80 pad 1: GND -> Net-(D1-Pad1)
- D80 pad 2: Net-(D74-Pad2) -> Net-(D80-Pad2)
- D81 pad 1: GND -> Net-(D1-Pad1)
- D81 pad 2: Net-(D74-Pad2) -> Net-(D81-Pad2)
- D82 pad 1: GND -> Net-(D1-Pad1)
- D82 pad 2: Net-(D74-Pad2) -> Net-(D82-Pad2)
- D83 pad 1: GND -> Net-(D1-Pad1)
- D83 pad 2: Net-(D74-Pad2) -> Net-(D83-Pad2)
- D84 pad 1: GND -> Net-(D1-Pad1)
- D84 pad 2: Net-(D74-Pad2) -> Net-(D84-Pad2)
- D85 pad 1: GND -> Net-(D1-Pad1)
- D85 pad 2: Net-(D74-Pad2) -> Net-(D85-Pad2)
- D86 pad 1: GND -> Net-(D1-Pad1)
- D86 pad 2: Net-(D74-Pad2) -> Net-(D86-Pad2)
- D87 pad 1: GND -> Net-(D1-Pad1)
- D87 pad 2: Net-(D74-Pad2) -> Net-(D87-Pad2)
- D9 pad 1: GND -> Net-(D1-Pad1)
- D9 pad 2: Net-(D1-Pad2) -> Net-(D9-Pad2)
- R1 pad 1: PWM -> Net-(D1-Pad2)
- R1 pad 2: Net-(D1-Pad2) -> VBUS
- R2 pad 1: PWM -> Net-(D2-Pad2)
- R2 pad 2: Net-(D16-Pad2) -> VBUS
- R3 pad 1: PWM -> Net-(D3-Pad2)
- R3 pad 2: Net-(D31-Pad2) -> VBUS
- R4 pad 1: PWM -> Net-(D4-Pad2)
- R4 pad 2: Net-(D46-Pad2) -> VBUS
- R5 pad 1: PWM -> Net-(D5-Pad2)
- R5 pad 2: Net-(D60-Pad2) -> VBUS
- R6 pad 1: PWM -> Net-(D6-Pad2)
- R6 pad 2: Net-(D74-Pad2) -> VBUS
- U1 pad 10: Col6 -> Col7
- U1 pad 11: Col5 -> Col6
- U1 pad 12: Col4 -> Col5
- U1 pad 14: Row0 -> Col4
- U1 pad 40: (no net) -> VBUS
- U1 pad 5: Col9 -> Row0
- U1 pad 6: Col8 -> Col9
- U1 pad 7: Col1 -> Col8
- U1 pad 9: Col7 -> Col1
Routing:
- net Net-(D1-Pad1): track 0.00 -> 2242.2 mm, vias 0 -> 66
- net VBUS: track 0.00 -> 1977.1 mm, vias 0 -> 69
- net Net-(D74-Pad2): track 407.5 -> 2.35 mm, vias 1 -> 0
- net Net-(D46-Pad2): track 377.8 -> 2.35 mm, vias 3 -> 0
- net Net-(D31-Pad2): track 365.0 -> 2.35 mm, vias 6 -> 0
- net Net-(D1-Pad2): track 340.1 -> 2.35 mm
- net Net-(D60-Pad2): track 302.2 -> 2.48 mm
- net Net-(D16-Pad2): track 298.7 -> 2.35 mm, vias 4 -> 0
- net PWM: track 222.2 -> 7.52 mm, vias 1 -> 0
- net Col5: track 469.2 -> 431.0 mm, vias 5 -> 2
- net Col4: track 438.0 -> 408.1 mm, vias 8 -> 9
- net Row6: track 229.8 -> 203.1 mm, vias 3 -> 12
- net Row0: track 293.0 -> 269.3 mm
- net Net-(D105-Pad1): track 127.6 -> 105.7 mm, vias 4 -> 5
- net Row8: track 203.2 -> 183.5 mm, vias 3 -> 10
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
Commit message: Mount Hall の位置を調節した。3D モデルには手を着けてないから使えないよ！
Parts:
- moved H14 6.98 mm to (301.0, 123.8)
- moved H9 6.98 mm to (331.5, 123.8)
- moved H8 5.12 mm to (394.3, 90.2)
- moved H2 3.81 mm to (331.5, 66.0)
- moved H15 2.84 mm to (331.5, 90.2)
- moved H11 0.63 mm to (331.5, 181.0)
- moved H12 0.63 mm to (146.1, 181.0)
- moved H3 0.63 mm to (222.2, 181.0)
- moved H6 0.63 mm to (394.3, 190.5)
Routing:
- net Col9: track 345.3 -> 353.5 mm, vias 2 -> 4
- net Col8: track 320.3 -> 323.4 mm
- net Row0: track 269.3 -> 271.5 mm
Other:
- board size 365.8 x 137.2 mm -> 366.4 x 137.2 mm

Commit message: GS間抵抗を追加。G抵抗を追加。なんかスイッチのフットプリント一つ消えちゃった
Parts:
- removed SW38: CherryMX, Button_Switch_Keyboard:SW_Cherry_MX_1.00u_PCB
- added C1: 3.3u, Capacitor_SMD:C_0603_1608Metric, B.Cu at (140.2, 64.0)
- added R89: 10k, Resistor_SMD:R_0603_1608Metric, B.Cu at (148.3, 90.4)
- R88: value 1k -> 100
- moved Q1 0.38 mm to (148.3, 93.3)
- moved R88 0.38 mm to (143.5, 92.5)
Connections:
- U1 pad 21: (no net) -> Net-(U1-Pad21)
- U1 pad 22: (no net) -> Net-(U1-Pad22)
- U1 pad 30: (no net) -> Net-(U1-Pad30)
- U1 pad 31: (no net) -> Net-(U1-Pad31)
- U1 pad 32: (no net) -> Net-(U1-Pad32)
- U1 pad 34: (no net) -> Net-(U1-Pad34)
- U1 pad 35: (no net) -> Net-(U1-Pad35)
- U1 pad 36: (no net) -> Net-(U1-Pad36)
- U1 pad 37: (no net) -> Net-(U1-Pad37)
- U1 pad 39: (no net) -> Net-(U1-Pad39)
Routing:
- net VBUS: track 1977.1 -> 2454.8 mm, vias 69 -> 15
- net Net-(D1-Pad1): track 2242.2 -> 2386.2 mm, vias 66 -> 18
- net Row4: track 276.1 -> 280.6 mm, vias 5 -> 2
- net Col9: track 353.5 -> 357.6 mm, vias 4 -> 1
- net Row1: track 187.1 -> 190.6 mm, vias 3 -> 0
- net Col0: track 284.8 -> 287.8 mm, vias 11 -> 0
- net Net-(Q1-Pad1): track 2.78 -> 0.00 mm
- net Row5: track 390.5 -> 388.4 mm, vias 5 -> 4
- net Row0: track 271.5 -> 271.6 mm, vias 2 -> 0
- net Row6: track 203.1 -> 203.0 mm, vias 12 -> 11
- net Col2: vias 8 -> 2
- net Col7: vias 3 -> 1
- net Row2: vias 5 -> 2
- net Net-(D105-Pad1): vias 5 -> 3
- net Col1: vias 3 -> 2
- removed copper zone on B.Cu, net GND
- removed copper zone on F.Cu, net GND

Commit message: Add files via upload
Parts:
- removed C1: 3.3u, Capacitor_SMD:C_0603_1608Metric
- removed R89: 10k, Resistor_SMD:R_0603_1608Metric
- added SW38: CherryMX, Button_Switch_Keyboard:SW_Cherry_MX_1.00u_PCB, F.Cu at (174.6, 123.8)
- R88: value 100 -> 1k
- moved Q1 0.38 mm to (148.0, 93.3)
- moved R88 0.38 mm to (143.5, 92.1)
Connections:
- U1 pad 21: Net-(U1-Pad21) -> (no net)
- U1 pad 22: Net-(U1-Pad22) -> (no net)
- U1 pad 30: Net-(U1-Pad30) -> (no net)
- U1 pad 31: Net-(U1-Pad31) -> (no net)
- U1 pad 32: Net-(U1-Pad32) -> (no net)
- U1 pad 34: Net-(U1-Pad34) -> (no net)
- U1 pad 35: Net-(U1-Pad35) -> (no net)
- U1 pad 36: Net-(U1-Pad36) -> (no net)
- U1 pad 37: Net-(U1-Pad37) -> (no net)
- U1 pad 39: Net-(U1-Pad39) -> (no net)
Routing:
- net VBUS: track 2454.8 -> 1977.1 mm, vias 15 -> 69
- net Net-(D1-Pad1): track 2386.2 -> 2242.2 mm, vias 18 -> 66
- net Row4: track 280.6 -> 276.1 mm, vias 2 -> 5
- net Col9: track 357.6 -> 353.5 mm, vias 1 -> 4
- net Row1: track 190.6 -> 187.1 mm, vias 0 -> 3
- net Col0: track 287.8 -> 284.8 mm, vias 0 -> 11
- net Net-(Q1-Pad1): track 0.00 -> 2.78 mm
- net Row5: track 388.4 -> 390.5 mm, vias 4 -> 5
- net Row0: track 271.6 -> 271.5 mm, vias 0 -> 2
- net Row6: track 203.0 -> 203.1 mm, vias 11 -> 12
- net Col2: vias 2 -> 8
- net Col7: vias 1 -> 3
- net Row2: vias 2 -> 5
- net Net-(D105-Pad1): vias 3 -> 5
- net Col1: vias 2 -> 3
- added copper zone on B.Cu, net GND
- added copper zone on F.Cu, net GND

Commit message: これからアンテナに気を付けつつベタグランドを追加する
Parts:
- renumbered SW1 to SWe
Routing:
- net Net-(D1-Pad1): track 2242.2 -> 2214.7 mm, vias 66 -> 19
- net VBUS: track 1977.1 -> 1999.6 mm, vias 69 -> 14
- net Col8: track 323.4 -> 327.5 mm, vias 3 -> 4
- net Col1: track 317.9 -> 313.9 mm, vias 3 -> 4
- net Col0: track 284.8 -> 288.6 mm, vias 11 -> 0
- net Row4: track 276.1 -> 273.4 mm, vias 5 -> 3
- net Row5: track 390.5 -> 393.2 mm, vias 5 -> 2
- net Col9: track 353.5 -> 353.4 mm, vias 4 -> 1
- net Row6: track 203.1 -> 203.0 mm, vias 12 -> 10
- net Col4: vias 9 -> 5
- net Col2: vias 8 -> 2
- net Row0: vias 2 -> 0
- net Col7: vias 3 -> 1
- net Row9: vias 9 -> 7
- net Row8: vias 10 -> 8
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- removed copper zone on B.Cu, net GND
- removed copper zone on F.Cu, net GND

Commit message: とりあえず配線幅を太くした。
Routing:
- net VBUS: track 1999.6 -> 2997.0 mm, vias 14 -> 16
- net Net-(D1-Pad1): track 2214.7 -> 3184.8 mm, vias 19 -> 20
- net Row4: track 273.4 -> 275.0 mm

Commit message: 配線の横に流れる電流値を記載しておいた。
Routing:
- net Net-(D1-Pad1): track 3184.8 -> 2988.6 mm, vias 20 -> 19
- net VBUS: track 2997.0 -> 2947.4 mm
- net Col8: track 327.5 -> 320.5 mm
Other:
- board text added: "114mA→"
- board text added: "120mA→"
- board text added: "228mA→"
- board text added: "243mA→"
- board text added: "261mA→"
- board text added: "39mA→"
- board text added: "78mA→"
- board text added: "99mA→"
- board text added: "←231mA"
- board text added: "←39mA"
- board text added: "←60mA"
- board text added: "←90mA"

Commit message: ベタグランドの配置途中
Routing:
- net VBUS: track 2947.4 -> 2957.7 mm
- net GND: vias 0 -> 64
- net (no net): vias 0 -> 9
- added copper zone on B.Cu, net GND
