File: pcb/circuit/circuit.kicad_pcb (KiCad board)
At the start: 2 copper layers, 366.4 x 137.2 mm, 366 parts, among them Q1 2N7002, SW1 CherryMX, SW10 CherryMX, SW11 CherryMX, SW12 CherryMX, SW13 CherryMX, SW14 CherryMX, SW15 CherryMX, SW16 CherryMX, SW17 CherryMX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

Commit message: PDF データでええやんってなった。
Routing:
- removed copper zone on B.Cu, net GND
- removed copper zone on F.Cu, net GND
